File: hardware/kicad/faff2_cbs1/test_debug.kicad_sch (KiCad schematic)
At the start: 0 parts

Commit message: mcu, test_debug: draw the MCU + USB + QSPI RAM and debug blocks
Fills the two block sheets this task owns. Nothing else in the KiCad
project is touched, and no MCU pin is re-assigned - the .ioc stays the
authority (DEC-0013) and was traced against the block diagram with no
conflict found.

mcu.kicad_sch
  - STM32H723VET6 across all six units, with DS13313 supply treatment:
    100nF per VDD pin plus a 4u7 bulk, 2x2u2 on VCAP (Table 14),
    2x100nF + 2x1uF on VDDA/VREF+, 100nF on NRST (Figure 18).
  - Boot and reset: 10k BOOT0 pull-down fitted, 1k pull-up DNP for DFU,
    reset button, hook test point, MCU_nRESET out to test_debug.
  - 24 MHz MEMS oscillator feeding both the STM32 HSE (external clock on
    PH0 only - PH1 is unallocated) and the USB3320 REFCLK, one 33R source
    termination per branch. This closes OQ-03.
  - USB3320C ULPI PHY in output-clock mode with its datasheet-mandated
    support parts (RBIAS 8k06 1%, RVBUS 10k device-only, REFSEL=111 for
    24 MHz, ID to VDD33, RESETB pull-down), a local 1.8 V LDO for VDD18
    - which the datasheet requires as a real external supply - and a 0R
    current break on the PHY 3.3 V rail.
  - USB-C receptacle, data only: 5.1k Rd on both CC lines, VBUS sensed
    through RVBUS rather than consumed, USBLC6-2P6 on the high-speed
    pair, shield to GND through a fitted 0R. The PHY sensing VBUS is why
    VBUS_MON (PC5) stays free for the motor DC link, supporting OQ-01.
  - OCTOSPI1 force-profile RAM: IS66WVS4M8BLL-104NLI, the 3.0 V part
    (ALL is the 1.8 V one), CE# pull-up, no series termination and no
    test points (DEC-0018 ruling 1).
  - MCO2 exposed as ADS1235_CLKIN; spare-I/O breakout header (DNP) so
    OQ-06 and OQ-07 can be served by a wire mod.

test_debug.kicad_sch
  - One header carrying SWD and USART3 (REQ-AR-15) in the standard ARM
    Cortex 10-pin order so a stock probe cable fits, with the console on
    the two KEY/NC positions through 100R series resistors.
  - Consolidated rail probe heade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
Parts:
- added J401: TSW-105-07-F-D, Amodo:TSW-105-07-F-D, symbol Amodo_Connectors:Header_Male_10-way_2-row_Straight_2.54mm_THT
- added J402: PH1-06-UA, Amodo:Adam_Tech_PH1-06-UA, symbol Amodo_Connectors:Header_Male_6-way_1-row_Straight_2.54mm_THT
- added R401, R402: 100R, Amodo:R_0603_1608Metric, symbol Amodo_Resistors:RES_TF_100R_0603
- added TP401, TP402, TP403, TP404, TP405, TP406: TestPoint, Amodo:KeystoneMiniatureTestLoop, symbol Amodo_Connectors:TestPointHook
Connections:
- new net: J401.7 (Pin_7), R401.1
- new net: J401.8 (Pin_8), R402.1
- new net +3V3: J401.1 (Pin_1), J402.2
- new net +3V3A: J402.3
- new net +5V: J402.1
- new net DBG_RX: R401.2
- new net DBG_TX: R402.2
- new net GND: J401.3 (Pin_3), J401.5 (Pin_5), J401.9 (Pin_9), J402.4, J402.5, J402.6, TP401.1, TP402.1, TP403.1, TP404.1, TP405.1, TP406.1
- new net MCU_nRESET: J401.10 (Pin_10)
- new net SWCLK: J401.4 (Pin_4)
- new net SWDIO: J401.2 (Pin_2)
- new net SWO: J401.6 (Pin_6)
Other:
- note added: "BLOCK: test_debug - system-level bring-up hardware that no functional block owns (DEC-0007). Everything here observes; nothing here generates a rail or a signal, so this sheet owns no isolation link or current break. Per-block test points, links and breaks stay in the sheet that produces the net. ROOT SHEET NEEDS - hierarchical labels this sheet exposes, all of them shared with the mcu block: SWD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"
- note added: "One header to check every logic rail with a DMM during bring-up steps 2 and 3 of TEST_PLAN 5. The rails themselves, and their isolation links and current breaks, belong to power_rails - this header only observes them. 1 +5V 2 +3V3 3 +3V3A 4 GND 5 GND 6 GND +24V IS DELIBERATELY NOT ON THIS HEADER. 24 V next to 3.3 V on a 2.54 mm strip is one slip away from destroying the board; power_entry_24v alr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"
- note added: "PINOUT - standard ARM Cortex Debug 10-pin order on 2.54 mm pitch, so a 2x5 SWD probe cable plugs straight on: 1 VTref (+3V3) 2 SWDIO 3 GND 4 SWCLK 5 GND 6 SWO 7 DBG_RX 8 DBG_TX 9 GND 10 nRESET Pins 7 and 8 are KEY / NC on the ARM pinout and are reused here for the USART3 console (REQ-AR-15 and the block diagram both put SWD and UART on ONE header). They are SWD-safe: an SWD probe drives only 2, 4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"
- note added: "SHEET NOTES"
- note added: "Six through-hole GND loops, spread across the board so an oscilloscope ground clip is never far from the signal hook being probed. The house standard asks for these wherever TestPointHook is used, and the block sheets use hooks on I2C1, SPI2, SPI3 and the fault lines."
- note added: "T1 DEBUG HEADER - SWD + USART3 CONSOLE (REQ-AR-15)"
- note added: "T2 CONSOLIDATED RAIL PROBE HEADER (TEST_PLAN 4)"
- note added: "T3 GND HOOKS FOR SCOPE CLIPS"
- note removed: "BLOCK: test_debug SCOPE System-level bring-up hardware that no single functional block owns. SWD debug connector (PA13 SWDIO, PA14 SWCLK, PB3 SWO), the USART3 debug console header (PD8 DBG_TX, PD9 DBG_RX), a consolidated rail probe header, and any cross-block isolation link that sits between two blocks rather than inside one. Per-block test points live in their own block sheets (DEC-0007). Bring-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"
