File: hardware/kicad/faff2_cbs1/motor_drive.kicad_sch (KiCad schematic)
At the start: 0 parts

Commit message: motor_drive: draw the DRV8323S gate driver, 3-phase stage and motor interface
Fills hardware/kicad/faff2_cbs1/motor_drive.kicad_sch: 24 V motor bus with
isolation link and current break, 210 uF bulk store, DC-link sense, DRV8323S
gate driver on SPI2, six BSZ099N06LS5 in a 3-phase bridge with 0R15 shunts,
phase-current conditioning into ADC1/2, power-stage NTC, and the motor and
rotary-encoder/hall connectors.

Closes OQ-08: the per-variant peak current limit (REQ-SF-03) needs no board
variant. One 0R15 shunt serves both builds; V50N uses CSA gain 5 V/V, where
+/-1.87 A full scale puts the 75 N (1.843 A) limit on the last ADC code, and
V10N uses gain 20 V/V. The DRV8323 VSENSE comparator (SEN_LVL 00b, 1.667 A =
67.8 N) is the hardware backstop, and every trip lands on nFAULT -> TIM1_BKIN.

The DRV8323S symbol is project-local (faff2_motor.kicad_sym); the Amodo house
library is read-only and is left untouched. Its footprint is deliberately
deferred - TI's current SLVSDJ3D PDF omits the RTA0040 package drawing.

Design record and the full Root sheet needs table:
docs/decisions/actuator-sch-motor.md

Co-Authored-By: Claude Opus 5 <noreply@anthropic.com>
Claude-Session: https://claude.ai/code/session_019CZNhkSJZhXK4S3Fzq8RKm
Parts:
- added C1101, C1102: 100uF, Amodo:C_ALU_D10_L10.2_SMT_ANTI-VIBE, symbol Amodo_Capacitors:CAP_ALU_100UF_SMD_20%_63V
- added C1103, C1110: 10uF, Amodo:C_1210_3225Metric, symbol Amodo_Capacitors:CAP_MLCC_10uF_1210_20%_63V
- added C1104, C1109: 100nF, Amodo:C_0805_2012Metric, symbol Amodo_Capacitors:CAP_MLCC_100nF_0805_10%_100V
- added C1105: 10nF, Amodo:C_0603_1608Metric, symbol Amodo_Capacitors:CAP_MLCC_10nF_0603_20%_50V
- added C1106, C1108, C1113: 100nF, Amodo:C_0402_1005Metric, symbol Amodo_Capacitors:CAP_MLCC_100nF_0402_10%_50V
- added C1107: 10uF, Amodo:C_0805_2012Metric, symbol Amodo_Capacitors:CAP_MLCC_10uF_0805_20%_25V
- added C1111: 1uF, Amodo:C_0603_1608Metric, symbol Amodo_Capacitors:CAP_MLCC_1uF_0603_10%_50V
- added C1112: 47nF, Amodo:C_0603_1608Metric, symbol Amodo_Capacitors:CAP_MLCC_47nF_0603_10%_50V
- added C1114, C1115: 1uF, Amodo:C_0603_1608Metric, symbol Amodo_Capacitors:CAP_MLCC_1uF_0603_10%_16V
- added C1116, C1117, C1118: 100pF, Amodo:C_0603_1608Metric, symbol Amodo_Capacitors:CAP_MLCC_100pF_0603_10%_50V
- added J1101, J1102: 1x6 2.54mm, Amodo:Adam_Tech_PH1-06-UA, symbol Amodo_Connectors:Header_Male_6-way_1-row_Straight_2.54mm_THT
- added J1103: Micro-Fit 1x3, Amodo:436500327, symbol Amodo_Connectors:Molex_Micro-Fit_3.0_Straight,1x3
- added Q1101, Q1102, Q1103, Q1104, Q1105, Q1106: BSZ099N06LS5, Amodo:PG-TSDSON-8-32, symbol Amodo_Power_Transistors:BSZ099N06LS5_AlternativeSym
- added R1101, R1102, R1114: 0R, Amodo:R_1206_3216Metric, symbol Amodo_Resistors:RES_TF_0R_1206_10A
- added R1103: 100k, Amodo:R_0603_1608Metric, symbol Amodo_Resistors:RES_TF_100k_0603
- added R1104: 12k, Amodo:R_0603_1608Metric, symbol Amodo_Resistors:RES_TF_12k_0603
- added R1105, R1111, R1112, R1113, R1115, R1118, R1120, R1121: 10k, Amodo:R_0603_1608Metric, symbol Amodo_Resistors:RES_TF_10k_0603
- added R1106, R1107, R1116, R1117, R1119: 0R, Amodo:R_0603_1608Metric, symbol Amodo_Resistors:RES_TF_0R_0603
- added R1108, R1109, R1110: 2k2, Amodo:R_0603_1608Metric, symbol Amodo_Resistors:RES_TF_2.2k_0603
- added R1122, R1123, R1124: 100R, Amodo:R_0603_1608Metric, symbol Amodo_Resistors:RES_TF_100R_0603
- added R1125, R1126, R1127: 0R15 5W, Amodo:R_4527_11470Metric, symbol Amodo_Resistors:RES_TF_0.15R_4527
- added RT1101: 10k NTC, Amodo:R_0603_1608Metric, symbol Amodo_Sensors:THERMISTOR_10k_0603
- added TP1101, TP1103, TP1104, TP1105, TP1106, TP1107, TP1108: TestPoint, Amodo:TestPoint_Pad_D1.0mm, symbol Amodo_Connectors:TestPoint
- added TP1102, TP1115, TP1118, TP1121: TestPoint, Amodo:TestPoint_Dual_D1.5mm_H1.0mm, symbol Amodo_Connectors:TestPointDual
- added TP1109, TP1110, TP1111, TP1112, TP1113, TP1114, TP1116, TP1117, TP1119, TP1120: TestPoint, Amodo:KeystoneMiniatureTestLoop, symbol Amodo_Connectors:TestPointHook
- added U1101: DRV8323S, symbol faff2_motor:DRV8323S
Connections:
- new net: Q1101.4 (G), TP1113.1, U1101.6 (GHA)
- new net: Q1106.1_2_3 (S_3), R1127.1, U1101.19 (SPC)
- new net: Q1106.4 (G), TP1120.1, U1101.18 (GLC)
- new net: R1123.1, TP1111.1, U1101.22 (SOB)
- new net: Q1104.1_2_3 (S_3), R1126.1, U1101.12 (SPB)
- new net: Q1104.4 (G), TP1117.1, U1101.13 (GLB)
- new net: Q1103.4 (G), TP1116.1, U1101.15 (GHB)
- new net: R1101.2, R1102.1
- new net: R1117.1, U1101.27 (SDI)
- new net: R1119.1, U1101.25 (nFAULT)
- new net: R1124.1, TP1112.1, U1101.21 (SOC)
- new net: Q1102.1_2_3 (S_3), R1125.1, U1101.9 (SPA)
- new net: Q1102.4 (G), TP1114.1, U1101.8 (GLA)
- new net: C1112.2, U1101.1 (CPL)
- new net: Q1105.4 (G), TP1119.1, U1101.16 (GHC)
- new net: C1112.1, U1101.2 (CPH)
- new net: R1122.1, TP1110.1, U1101.23 (SOA)
- new net: R1116.1, U1101.28 (SCLK)
- new net: C1111.2, TP1107.1, U1101.3 (VCP)
- new net: C1115.1, U1101.33 (DVDD)
- new net +24V_SW: R1101.1
- new net +3V3: C1113.1, C1114.1, R1105.1, R1106.1, R1108.1, R1109.1, R1110.1, R1111.1, R1112.1, R1113.1, R1115.1, R1118.1, R1120.1, U1101.24 (VREF)
- new net +5V: R1107.1
- new net CONFIG_SPI_MISO: R1118.2, U1101.26 (SDO)
- new net CONFIG_SPI_MOSI: R1117.2
- new net CONFIG_SPI_SCK: R1116.2
- new net DRV8323_CAL: U1101.31 (CAL)
- new net DRV8323_EN: R1121.1, U1101.30 (ENABLE)
- new net DRV8323_nCS: R1115.2, U1101.29 (nSCS)
- new net DRV8323_nFAULT: R1119.2, R1120.2, TP1109.1
- new net GND: C1101.2, C1102.2, C1103.2, C1104.2, C1105.2, C1106.2, C1107.2, C1108.2, C1109.2, C1110.2, C1113.2, C1114.2, C1115.2, C1116.2, C1117.2, C1118.2, J1101.5, J1101.6, J1102.5, J1102.6, R1104.2, R1121.2, R1125.2, R1126.2, R1127.2, RT1101.2, TP1102.2, TP1108.1, TP1115.2, TP1118.2, TP1121.2, U1101.10 (SNA), U1101.11 (SNB), U1101.20 (SNC), U1101.32 (AGND), U1101.40 (PGND), U1101.41 (PAD)
- new net HALL1: J1102.2, R1111.2
- new net HALL2: J1102.3, R1112.2
- new net HALL3: J1102.4, R1113.2
- new net MOTOR_ENCODER_A: J1101.2, R1108.2
- new net MOTOR_ENCODER_B: J1101.3, R1109.2
- new net MOTOR_ENCODER_I: J1101.4, R1110.2
- new net MOTOR_FETTEMP: C1106.1, R1105.2, RT1101.1, TP1104.1
- new net MOTOR_I_A: C1116.1, R1122.2
- new net MOTOR_I_B: C1117.1, R1123.2
- new net MOTOR_I_C: C1118.1, R1124.2
- new net MOTOR_PWM_AH: U1101.34 (INHA)
- new net MOTOR_PWM_AL: U1101.35 (INLA)
- new net MOTOR_PWM_BH: U1101.36 (INHB)
- new net MOTOR_PWM_BL: U1101.37 (INLB)
- new net MOTOR_PWM_CH: U1101.38 (INHC)
- new net MOTOR_PWM_CL: U1101.39 (INLC)
- new net MOTOR_U: J1103.1, Q1101.1_2_3 (S_3), Q1102.5_6_7_8 (D_2), TP1115.1, U1101.7 (SHA)
- new net MOTOR_V: J1103.2, Q1103.1_2_3 (S_3), Q1104.5_6_7_8 (D_2), TP1118.1, U1101.14 (SHB)
- new net MOTOR_W: J1103.3, Q1105.1_2_3 (S_3), Q1106.5_6_7_8 (D_2), TP1121.1, U1101.17 (SHC)
- new net V24_MOT: C1101.1, C1102.1, C1103.1, C1104.1, Q1101.5_6_7_8 (D_2), Q1103.5_6_7_8 (D_2), Q1105.5_6_7_8 (D_2), R1102.2, R1103.1, R1114.1, TP1101.1, TP1102.1, U1101.5 (VDRAIN)
- new net VBUS_MON: C1105.1, R1103.2, R1104.1, TP1103.1
- new net VENC: C1107.1, C1108.1, J1101.1, J1102.1, R1106.2, R1107.2, TP1105.1
- new net VM_DRV: C1109.1, C1110.1, C1111.1, R1114.2, TP1106.1, U1101.4 (VM)
Other:
- note added: "24 V MOTOR BUS, BULK STORE AND DC-LINK SENSE"
- note added: "3-PHASE POWER STAGE AND PHASE-CURRENT SHUNTS"
- note added: "Bulk store 210 uF; DC-link ripple < 0.15 V at 1.9 A, 20 kHz. VBUS_MON 100k/12k: 3.30 V full scale = 30.8 V bus; 24.0 V reads 2.571 V. PC5 / ADC2_INP8 (DEC-0011, OQ-01)."
- note added: "DESIGN NOTES"
- note added: "Encoder supply - FIT ONE ONLY. R1106 fitted = 3V3 (CALC budget). R1107 = 5 V read-head option. Pull-ups always go to 3V3, so the MCU never sees 5 V from an open- collector encoder or hall output."
- note added: "GATE DRIVER - DRV8323S (SPI)"
- note added: "J102 A/B/Z -> TIM3 CH1/CH2/CH3 (PC6/PC7/PC8). J103 halls -> PE14/PD14/PD15 (GPIO). Motor not fixed (DEC-0004): this pinout suits every candidate BLDC in the design log."
- note added: "MOTOR ROTARY ENCODER AND HALL SENSORS"
- note added: "POWER-STAGE TEMPERATURE"
- note added: "R101 isolation link, R102 current-measurement break. Both fitted. Opening R101 leaves the whole logic side powered with the actuator dead - TEST_PLAN.md 3.3, step 8."
- note added: "R1201 isolates the gate-driver supply from the motor bus. VDRAIN comes from the high-side FET drains, not from VM, so the VDS monitor sees the real bridge rail (SLVSDJ3D 11.1)."
- note added: "RT1101 sits on the power stage, between the low-side FETs. 10k NTC, B = 3435 K, 10k pull-up: 1.65 V at 25 C, 0.86 V at 85 C. PA4 / ADC1_INP18 (DEC-0011)."
- note added: "SAFETY-CRITICAL BREAK PATH. R1206 is FITTED by default and marked on the silkscreen. DRV8323_nFAULT (open drain) drives TIM1_BKIN on PE15; opening R1206 exercises the LIMIT_nBRK path alone (TEST_PLAN.md 3.3, bring-up step 8). R1207 holds PE15 high while R1206 is out. R1203/R1204 are the SPI2 stub links - remove both to lift U1101 off the shared bus; SDO is open drain and Hi-Z while nSCS is high, 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"
- note added: "TIM1 CH1/CH1N..CH3/CH3N (PE8-PE13), 6x PWM mode, dead time in the MCU. INHx/INLx have internal 100k pull-downs; ENABLE low forces GHx to SHx and GLx to PGND, so the bridge is off in MCU reset."
- note added: "VREF ties the CSA reference to the same +3V3 the STM32 ADC uses, so phase current is ratiometric. DVDD is the DRV internal 3.3 V regulator: decoupling only, no load."
- note removed: "BLOCK: motor_drive SCOPE 3-phase inverter for a 24 V BLDC. DRV8323 SPI-variant gate driver (per the .ioc nets DRV8323_nCS/EN/CAL/nFAULT) with its three integrated current-sense amplifiers, six power FETs, DC-link sense and bulk capacitance, motor phase connector, FET temperature sense, and the motor rotary encoder / Hall sensor interface (DEC-0004). Peak current sense limit is configurable per va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"
- title: CBs_1 - Motor Drive (DRV8323) -> CBs_1 - Motor Drive (DRV8323S)

Commit message: motor_drive: correct the designators quoted in the sheet notes and the record
Designators are allocated in placement order, so the numbers written into the
on-sheet notes and docs/decisions/actuator-sch-motor.md by hand were wrong: the
shunts are R1125-R1127 not R1301-R1303, the break-path link is R1119, and the
motor phase connector is J1103. Every designator the record quotes now exists
on the sheet.

Co-Authored-By: Claude Opus 5 <noreply@anthropic.com>
Claude-Session: https://claude.ai/code/session_019CZNhkSJZhXK4S3Fzq8RKm
Other:
- note added: "R1114 isolates the gate-driver supply from the motor bus. VDRAIN comes from the high-side FET drains, not from VM, so the VDS monitor sees the real bridge rail (SLVSDJ3D 11.1)."
- note added: "SAFETY-CRITICAL BREAK PATH. R1119 is FITTED by default and marked on the silkscreen. DRV8323_nFAULT (open drain) drives TIM1_BKIN on PE15; opening R1119 exercises the LIMIT_nBRK path alone (TEST_PLAN.md 3.3, bring-up step 8). R1120 holds PE15 high while R1119 is out. R1116/R1117 are the SPI2 stub links - remove both to lift U1101 off the shared bus; SDO is open drain and Hi-Z while nSCS is high, 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"
- note removed: "R1201 isolates the gate-driver supply from the motor bus. VDRAIN comes from the high-side FET drains, not from VM, so the VDS monitor sees the real bridge rail (SLVSDJ3D 11.1)."
- note removed: "SAFETY-CRITICAL BREAK PATH. R1206 is FITTED by default and marked on the silkscreen. DRV8323_nFAULT (open drain) drives TIM1_BKIN on PE15; opening R1206 exercises the LIMIT_nBRK path alone (TEST_PLAN.md 3.3, bring-up step 8). R1207 holds PE15 high while R1206 is out. R1203/R1204 are the SPI2 stub links - remove both to lift U1101 off the shared bus; SDO is open drain and Hi-Z while nSCS is high, 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"
Changed lines of the file:
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@@
 		)
 	)
-	(text "R1201 isolates the gate-driver\nsupply from the motor bus.\nVDRAIN comes from the high-side\nFET drains, not from VM, so the\nVDS monitor sees the real bridge\nrail (SLVSDJ3D 11.1)."
+	(text "R1114 isolates the gate-driver\nsupply from the motor bus.\nVDRAIN comes from the high-side\nFET drains, not from VM, so the\nVDS monitor sees the real bridge\nrail (SLVSDJ3D 11.1)."
 		(exclude_from_sim no)
 		(at 195.58 22.86 0)
@@
 		)
 	)
-	(text "SAFETY-CRITICAL BREAK PATH. R1206 is FITTED by default and marked on the silkscreen. DRV8323_nFAULT (open drain) drives\nTIM1_BKIN on PE15; opening R1206 exercises the LIMIT_nBRK path alone (TEST_PLAN.md 3.3, bring-up step 8). R1207 holds PE15\nhigh while R1206 is out. R1203/R1204 are the SPI2 stub links - remove both to lift U1101 off the shared bus; SDO is open\ndrain and Hi-Z while nSCS is high, so MISO needs no link. R1208 keeps ENABLE - and the bridge - off until PD10 drives high.\n\nPEAK CURRENT LIMIT (REQ-SF-03, closes OQ-08). One shunt value serves both variants; the limit is an SPI setting plus a\nfirmware threshold, not a board change. 0R15 with CSA gain 5 V/V gives +/-1.87 A full scale on V50N, so the 75 N (1.843 A)\nlimit lands on the last ADC code; gain 20 V/V gives +/-0.467 A on V10N, 15 N at 79 % of scale. SEN_LVL 00b trips the\nhardware comparator at 1.667 A = 67.8 N, below the V50N cell limit. A V10N build wanting that trip at 15 N fits 0R68.\n\nPOWER STAGE. No series gate resistors and no G-S pull-downs - slew rate is set by IDRIVE/TDRIVE over SPI, and external\ngate parts degrade the VDS and gate-fault monitors. SPx is the VDS monitor return as well as the CSA input, so keep it\nKelvin to the FET source. LAYOUT: shunt -> PGND -> bulk-cap negative is ONE tight loop, joined to system ground at a\nsingle point at the bulk capacitors."
+	(text "SAFETY-CRITICAL BREAK PATH. R1119 is FITTED by default and marked on the silkscreen. DRV8323_nFAULT (open drain) drives\nTIM1_BKIN on PE15; opening R1119 exercises the LIMIT_nBRK path alone (TEST_PLAN.md 3.3, bring-up step 8). R1120 holds PE15\nhigh while R1119 is out. R1116/R1117 are the SPI2 stub links - remove both to lift U1101 off the shared bus; SDO is open\ndrain and Hi-Z while nSCS is high, so MISO needs no link. R1121 keeps ENABLE - and the bridge - off until PD10 drives high.\n\nPEAK CURRENT LIMIT (REQ-SF-03, closes OQ-08). One shunt value serves both variants; the limit is an SPI setting plus a\nfirmware threshold, not a board change. 0R15 with CSA gain 5 V/V gives +/-1.87 A full scale on V50N, so the 75 N (1.843 A)\nlimit lands on the last ADC code; gain 20 V/V gives +/-0.467 A on V10N, 15 N at 79 % of scale. SEN_LVL 00b trips the\nhardware comparator at 1.667 A = 67.8 N, below the V50N cell limit. A V10N build wanting that trip at 15 N fits 0R68.\n\nPOWER STAGE. No series gate resistors and no G-S pull-downs - slew rate is set by IDRIVE/TDRIVE over SPI, and external\ngate parts degrade the VDS and gate-fault monitors. SPx is the VDS monitor return as well as the CSA input, so keep it\nKelvin to the FET source. LAYOUT: shunt -> PGND -> bulk-cap negative is ONE tight loop, joined to system ground at a\nsingle point at the bulk capacitors."
 		(exclude_from_sim no)
 		(at 251.46 222.25 0)

Commit message: integrate: wire the root sheet - 113 sheet pins, 70 wires, ERC 0/0
Closes DEC-0009. Every net that crosses a block boundary is now drawn on
the root sheet: one sheet pin per hierarchical label a child declares,
each on a wire. Nothing on the root connects by name.

The layout is the block diagram of docs/FAFF-2-Electronics-Full.svg read
left to right - 24 V in top left, sensing and user I/O down the left
column, the MCU in the middle, motor drive on the right. Each peer
block's pin rows are aligned with the mcu rows they face, so all 48
mcu-to-peer nets are single straight wires with no bends and no
crossings.

Two topologies needed care:

  * power_entry_24v fans out to three different places. Its pins sit on
    a 5.08 mm pitch and the three routes are nested - V24_LOGIC straight
    across to power_rails, +24V_SW peeling down and running over the top
    of the mcu block to motor_drive, V24_MON dropping inside it - so no
    two cross.
  * the shared SPI2 CONFIG bus is tapped once per wire between
    motor_drive and temp_sense, which is why temp_sense sits under
    motor_drive rather than in the sensor column. The three taps and the
    ADS1120_nCS run are nested the same way: four junctions, zero
    crossings.

motor_drive declared CONFIG_SPI_MISO an output while temp_sense declared
it tri_state - the reconciliation actuator-sch-afe.md asked for at
integration. Both are tri_state now: three devices share that wire and
each drives it only while its own chip select is low.

Verification, whole project, nothing suppressed:
  ERC --severity-all          0 errors, 0 warnings (was 194 violations)
  netlist                     409 components, no duplicate references,
                              311 -> 253 nets, exactly the 58 merges the
                              113 pins over 55 net names predict
  overlap checker             root sheet clean; the 11 findings left in
                              linear_encoder / loadcell_afe / temp_sense
                     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
Changed lines of the file:
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@@
 	)
 	(hierarchical_label "CONFIG_SPI_MISO"
-		(shape output)
+		(shape tri_state)
 		(at 137.16 168.91 180)
 		(effects

Commit message: integrate: RTA0040B land pattern for the DRV8323S, and two footprints assigned
The DRV8323S footprint was owed since the motor block landed: SLVSDJ3D
ships the RTV0032E and RGZ0048A package drawings but not RTA0040's, so
there was nothing to draw from.

Found it: TI drawing 4219112/A (07/2018), RTA0040B, in the DRV8353 data
sheet pp.98-100. Committed as
datasheets/DRV832x_RTA0040B_package_4219112A.pdf so the next reader does
not repeat the hunt. Set beside TI 4219052/A (RHA0040B, from
msp430g2755.pdf p.72), the two give an identical outline and an identical
land pattern - 6.1/5.9 body, 36X 0.5 pitch, 2X 4.5 terminal span, 40X
0.5/0.3 terminal length, 4.15+/-0.1 exposed pad, land 40X (0.6)x(0.22)
inside (5.8), stencil 9X (1.17) on (1.37) - and differ only in package
height, 0.8 mm WQFN against 1.0 mm VQFN.

So KiCad 9's official Texas_RHA0040B footprint is a dimension-verified
base, which is what pcb-layout-style allows: its perimeter pads,
silkscreen, fab outline and courtyard are reproduced in
faff2.pretty/Texas_RTA0040B_WQFN-40-1EP_6x6mm_P0.5mm_EP4.15x4.15mm, with
two deliberate departures - TI's own 9X (1.17) on (1.37) stencil
apertures (71.5% coverage against TI's stated 71%), and IPC-nominal
perimeter pads kept as a superset of TI's own tighter land, matching the
house QFN footprints in Amodo.pretty and leaving an inspectable toe.

Geometry asserted programmatically: 40 pads, ten a side, 0.5 mm pitch,
4.5 mm span, row offset 2.9375, EP 4.15 square, pin 1 the top pad of the
left column - the anticlockwise numbering of SLVSDJ3D figure 6-6, which
the symbol's own 41 pins (pin 41 = PAD) match name for name.

U601 (AM26LV32, linear_encoder) also had no footprint: the house
AM26LS32Ax symbol carries none. Assigned Amodo:SOIC-16-N, the reviewed
house land for the 3.9x9.9 mm D package the part's mpn names. Every one
of the 409 components now resolves to a footprint, and all 51 distinct
footprints resolve to a file in Amodo.pretty or faff2.pretty.

ERC still 0/0 at seve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
Parts:
- U1101: footprint (none) -> faff2:Texas_RTA0040B_WQFN-40-1EP_6x6mm_P0.5mm_EP4.15x4.15mm
Changed lines of the file:
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@@
 			)
 		)
-		(property "Footprint" ""
+		(property "Footprint" "faff2:Texas_RTA0040B_WQFN-40-1EP_6x6mm_P0.5mm_EP4.15x4.15mm"
 			(at 218.44 123.19 0)
 			(effects
