File: hardware/kicad/faff2_cbs1/temp_sense.kicad_sch (KiCad schematic)
At the start: 44 parts, among them J701 1752120, J702 1752120, U701 ADS1120

Commit message: review r1: logic-analyser headers, U501 reference note, AFE/encoder fixes
Answers the captain's round-1 review points on loadcell_afe, linear_encoder,
temp_sense and nvm_calibration.

U501 and the reference (R1). The ADS1235 has no internal reference and no
reference output pin - REFP0/REFN0 are inputs. The reference is the load cell's
own excitation, sensed at the bridge, which is what makes the measurement
ratiometric. Documented in a 15-line note beside U501B's reference pins.

Logic-analyser headers (R2, R5). The Amodo keyed 10-way 0.1in socket
(8510-4500PL) replaces the per-net hooks:

  J502  loadcell_afe   CH0..CH7 = the whole SPI3 interface plus nDRDY, START,
                       nRESET and CLKIN; TP506..TP512 and TP514 removed
  J603  linear_encoder CH0..CH4 = the three receiver outputs plus ENC_SDO and
                       ENC_nPROG; TP602..TP607 removed

Both tap the driver side of the series terminators, so the header still sees the
bus when an isolation link is lifted. J602 is KEPT: it carries REQ-PS-09, its
pin 9 is +5V_ENC where the socket wants GND, and six of its signals are the
terminated RS-422 pairs that DEC-0018 ruling 1 keeps stub-free. Raised as a
decision; ruled option (a) and captain-ratified.

J601 (R3, R4). Reference text moved off the body; the project-local
FH12-10S-0.5SH(55) symbol now shows pin numbers and names every pin (1..10,
MP1/MP2), matching the FH35C house exemplar. Fixed in faff2_periph.kicad_sym
and in the sheet's embedded copy, so no lib_symbol_mismatch.

5 V read-head supply (R6). R608, R609 and D602 are DNP parallel positions on
R601, FB601 and D601. Not for current sharing - the ferrite alone has 4x margin
on the CALC budget - but for bring-up: a shunt at R608 meters head current in
circuit, R609 bypasses the bead, D602 is a second SC-79 clamp. Moving D601 up
to make room also cleared its value text off the ENC_nPROG label and its ground
triangle off the ENC_nPROG wire.

temp_sense C701/C702 (R7). Both had their groun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
Connections:
- net GND: now also C701.2, C702.2; no longer C701.1, C702.1
- net at C703.2, R702.2, U701.10 (AIN1): now also C702.1; no longer C702.2
- net at C703.1, R701.2, U701.11 (AIN0/REFP1): now also C701.1; no longer C701.2
Other:
- moved on the sheet: C701, C702
Changed lines of the file:
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@@
 	(symbol
 		(lib_id "Amodo_Capacitors:CAP_MLCC_10nF_0603_5%_100V")
-		(at 109.22 17.78 0)
+		(at 109.22 35.56 0)
 		(unit 1)
 		(exclude_from_sim no)
@@
 		(dnp no)
 		(property "Reference" "C701"
-			(at 111.51 17.14 0)
+			(at 111.51 34.92 0)
 			(do_not_autoplace yes)
 			(effects
@@
 		)
 		(property "Value" "10nF"
-			(at 111.51 19.05 0)
+			(at 111.51 36.83 0)
 			(do_not_autoplace yes)
 			(effects
@@
 		)
 		(property "Footprint" "Amodo:C_0603_1608Metric"
-			(at 109.22 17.78 0)
+			(at 109.22 35.56 0)
 			(do_not_autoplace yes)
 			(effects
@@
 		)
 		(property "Datasheet" "https://product.tdk.com/system/files/dam/doc/product/capacitor/ceramic/mlcc/catalog/mlcc_automotive_esd_en.pdf"
-			(at 109.22 17.78 0)
+			(at 109.22 35.56 0)
 			(do_not_autoplace yes)
 			(effects
@@
 		)
 		(property "Description" "SMD MLCC Capacitor 10nF 0603 5% C0G 100V"
-			(at 109.22 17.78 0)
+			(at 109.22 35.56 0)
 			(do_not_autoplace yes)
 			(effects
@@
 		)
 		(property "mpn" "CGA3EAC0G2A103J080AC"
-			(at 109.22 17.78 0)
+			(at 109.22 35.56 0)
 			(do_not_autoplace yes)
 			(effects
@@
 		)
 		(property "SymLifecycle" "reviewed"
-			(at 109.22 17.78 0)
+			(at 109.22 35.56 0)
 			(do_not_autoplace yes)
 			(effects
@@
 	(symbol
 		(lib_id "Amodo_Symbols:GND")
-		(at 109.22 15.24 0)
+		(at 109.22 38.1 0)
 		(unit 1)
 		(exclude_from_sim no)
@@
 		(dnp no)
 		(property "Reference" "#PWR704"
-			(at 111.76 13.97 0)
+			(at 111.76 36.83 0)
 			(do_not_autoplace yes)
 			(effects
@@
 		)
 		(property "Value" "GND"
-			(at 111.76 16.51 0)
+			(at 111.76 39.37 0)
 			(do_not_autoplace yes)
 			(effects
@@
 		)
 		(property "Footprint" ""
-			(at 109.22 15.24 0)
+			(at 109.22 38.1 0)
 			(do_not_autoplace yes)
 			(effects
@@
 		)
 		(property "Datasheet" ""
-			(at 109.22 15.24 0)
+			(at 109.22 38.1 0)
 			(do_not_autoplace yes)
 			(effects
@@
 		)
 		(property "Description" "Power symbol creates a global label with name \"GND\" , ground"
-			(at 109.22 15.24 0)
+			(at 109.22 38.1 0)
 			(do_not_autoplace yes)
 			(effects
@@
 		)
 		(property "SymLifecycle" "tested"
-			(at 109.22 15.24 0)
+			(at 109.22 38.1 0)
 			(do_not_autoplace yes)
 			(effects
@@
 	(symbol
 		(lib_id "Amodo_Capacitors:CAP_MLCC_10nF_0603_5%_100V")
-		(at 119.38 17.78 0)
+		(at 119.38 35.56 0)
 		(unit 1)
 		(exclude_from_sim no)
@@
 		(dnp no)
 		(property "Reference" "C702"
-			(at 121.67 17.14 0)
+			(at 121.67 34.92 0)
 			(do_not_autoplace yes)
 			(effects
@@
 		)
 		(property "Value" "10nF"
-			(at 121.67 19.05 0)
+			(at 121.67 36.83 0)
 			(do_not_autoplace yes)
 			(effects
@@
 		)
 		(property "Footprint" "Amodo:C_0603_1608Metric"
-			(at 119.38 17.78 0)
+			(at 119.38 35.56 0)
 			(do_not_autoplace yes)
 			(effects
@@
 		)
 		(property "Datasheet" "https://product.tdk.com/system/files/dam/doc/product/capacitor/ceramic/mlcc/catalog/mlcc_automotive_esd_en.pdf"
-			(at 119.38 17.78 0)
+			(at 119.38 35.56 0)
 			(do_not_autoplace yes)
 			(effects
@@
 		)
 		(property "Description" "SMD MLCC Capacitor 10nF 0603 5% C0G 100V"
-			(at 119.38 17.78 0)
+			(at 119.38 35.56 0)
 			(do_not_autoplace yes)
 			(effects
@@
 		)
 		(property "mpn" "CGA3EAC0G2A103J080AC"
-			(at 119.38 17.78 0)
+			(at 119.38 35.56 0)
 			(do_not_autoplace yes)
 			(effects
@@
 		)
 		(property "SymLifecycle" "reviewed"
-			(at 119.38 17.78 0)
+			(at 119.38 35.56 0)
 			(do_not_autoplace yes)
 			(effects
@@
 	(symbol
 		(lib_id "Amodo_Symbols:GND")
-		(at 119.38 15.24 0)
+		(at 119.38 38.1 0)
 		(unit 1)
 		(exclude_from_sim no)
@@
 		(dnp no)
 		(property "Reference" "#PWR705"
-			(at 121.92 13.97 0)
+			(at 121.92 36.83 0)
 			(do_not_autoplace yes)
 			(effects
@@
 		)
 		(property "Value" "GND"
-			(at 121.92 16.51 0)
+			(at 121.92 39.37 0)
 			(do_not_autoplace yes)
 			(effects
@@
 		)
 		(property "Footprint" ""
-			(at 119.38 15.24 0)
+			(at 119.38 38.1 0)
 			(do_not_autoplace yes)
 			(effects
@@
 		)
 		(property "Datasheet" ""
-			(at 119.38 15.24 0)
+			(at 119.38 38.1 0)
 			(do_not_autoplace yes)
 			(effects
@@
 		)
 		(property "Description" "Power symbol creates a global label with name \"GND\" , ground"
-			(at 119.38 15.24 0)
+			(at 119.38 38.1 0)
 			(do_not_autoplace yes)
 			(effects
@@
 		)
 		(property "SymLifecycle" "tested"
-			(at 119.38 15.24 0)
+			(at 119.38 38.1 0)
 			(do_not_autoplace yes)
 			(effects
@@
 	(wire
 		(pts
-			(xy 109.22 22.86) (xy 109.22 20.32)
+			(xy 109.22 22.86) (xy 109.22 33.02)
 		)
 		(stroke
@@
 	(wire
 		(pts
-			(xy 119.38 27.94) (xy 119.38 20.32)
+			(xy 119.38 27.94) (xy 119.38 33.02)
 		)
 		(stroke

Commit message: review r1 final sweep: power labels, TP silkscreen names, text overlaps
The captain's design-wide pass, run once the per-sheet batches had landed.
Presentation only: ERC 0 errors / 0 warnings at severity-all, 404 components,
251 nets, and every per-net node set identical to the pre-sweep export.

  power labels   92 rail names were hidden on loadcell_afe, motor_drive and
                 temp_sense - all 285 power symbols now read, placed to the
                 house pattern (GND below the symbol, rail arrows above)
  test points    66 of 83 still carried the library default "TestPoint". All
                 83 now name what they measure, from the net they actually
                 land on in the netlist; longest is 5 characters
  text overlap   16 collisions cleared design-wide, four of them sub-millimetre
                 ones the bundled checker passes because it under-measures text
  GND upside down  none - 0 of 285 power symbols is rotated or mirrored
  graphic/wire   one: power_rails block D's bottom border lay along the last
                 PWR_FLAG's wire; the flag column moved up 2.54

The overlap checker turns out to have three separable blind spots, each settled
here by measuring a render rather than by reading the format: it grows every
text field rightward regardless of justify/mirror/180-rotation, so its box is a
mirror image of the truth for those and it both invents and misses collisions;
it measures text at ~1.06 mm per character where the real advance is ~1.19; and
it reflects a rotated symbol's body about the origin. tools/sch_geom.py models
all three correctly and the design is clean under it design-wide. Two of that
model's own rules - notes growing up from their anchor, and labels taking no
180-degree justify flip - were bugs of mine that the checker caught first. The
render is what settles it; neither tool is authoritative alone.

Placement is searched rather than guessed: 177 newly visible fields are tried
against every wire, block border, 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
Parts:
- TP701: value TestPoint -> PRB1A
- TP702: value TestPoint -> PRB1B
- TP703: value TestPoint -> PRB2A
- TP704: value TestPoint -> PRB2B
- TP705: value TestPoint -> REFP
- TP706: value TestPoint -> REFN
- TP707: value TestPoint -> DRDY
- TP708: value TestPoint -> nCS
- TP709: value TestPoint -> SCK
- TP710: value TestPoint -> MOSI
- TP711: value TestPoint -> MISO
- TP712, TP713: value TestPoint -> GND
Changed lines of the file:
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@@
 		)
 		(property "Value" "GND"
-			(at 73.66 44.45 0)
+			(at 71.12 48.26 0)
 			(do_not_autoplace yes)
 			(effects
@@
 					(size 1.27 1.27)
 				)
-				(justify left)
-				(hide yes)
 			)
 		)
@@
 		)
 		(property "Value" "GND"
-			(at 73.66 113.03 0)
+			(at 71.12 116.84 0)
 			(do_not_autoplace yes)
 			(effects
@@
 					(size 1.27 1.27)
 				)
-				(justify left)
-				(hide yes)
 			)
 		)
@@
 			)
 		)
-		(property "Value" "TestPoint"
-			(at 77.47 18.42 0)
+		(property "Value" "PRB1A"
+			(at 74.93 18.91 0)
 			(do_not_autoplace yes)
 			(effects
@@
 					(size 1.27 1.27)
 				)
-				(justify left)
-				(hide yes)
+				(justify right)
 			)
 		)
@@
 			)
 		)
-		(property "Value" "TestPoint"
-			(at 87.63 27.85 0)
+		(property "Value" "PRB1B"
+			(at 87.63 21.14 0)
 			(do_not_autoplace yes)
 			(effects
@@
 				)
 				(justify right)
-				(hide yes)
 			)
 		)
@@
 			)
 		)
-		(property "Value" "TestPoint"
-			(at 77.47 87 0)
+		(property "Value" "PRB2A"
+			(at 74.93 87.49 0)
 			(do_not_autoplace yes)
 			(effects
@@
 					(size 1.27 1.27)
 				)
-				(justify left)
-				(hide yes)
+				(justify right)
 			)
 		)
@@
 			)
 		)
-		(property "Value" "TestPoint"
-			(at 87.63 96.43 0)
+		(property "Value" "PRB2B"
+			(at 87.63 89.72 0)
 			(do_not_autoplace yes)
 			(effects
@@
 				)
 				(justify right)
-				(hide yes)
 			)
 		)
@@
 		)
 		(property "Value" "GND"
-			(at 91.44 128.27 0)
+			(at 88.9 130.81 0)
 			(do_not_autoplace yes)
 			(effects
@@
 					(size 1.27 1.27)
 				)
-				(justify left)
-				(hide yes)
 			)
 		)
@@
 		)
 		(property "Value" "GND"
-			(at 111.76 39.37 0)
+			(at 109.22 41.91 0)
 			(do_not_autoplace yes)
 			(effects
@@
 					(size 1.27 1.27)
 				)
-				(justify left)
-				(hide yes)
 			)
 		)
@@
 		)
 		(property "Value" "GND"
-			(at 121.92 39.37 0)
+			(at 119.38 41.91 0)
 			(do_not_autoplace yes)
 			(effects
@@
 					(size 1.27 1.27)
 				)
-				(justify left)
-				(hide yes)
 			)
 		)
@@
 		)
 		(property "Value" "GND"
-			(at 111.76 113.03 0)
+			(at 109.22 115.57 0)
 			(do_not_autoplace yes)
 			(effects
@@
 					(size 1.27 1.27)
 				)
-				(justify left)
-				(hide yes)
 			)
 		)
@@
 		)
 		(property "Value" "GND"
-			(at 121.92 113.03 0)
+			(at 121.92 115.57 0)
 			(do_not_autoplace yes)
 			(effects
@@
 				)
 				(justify left)
-				(hide yes)
 			)
 		)
@@
 		)
 		(property "Value" "GND"
-			(at 111.76 135.89 0)
+			(at 109.22 143.51 0)
 			(do_not_autoplace yes)
 			(effects
@@
 					(size 1.27 1.27)
 				)
-				(justify left)
-				(hide yes)
 			)
 		)
@@
 		)
 		(property "Value" "GND"
-			(at 121.92 135.89 0)
+			(at 119.38 143.51 0)
 			(do_not_autoplace yes)
 			(effects
@@
 					(size 1.27 1.27)
 				)
-				(justify left)
-				(hide yes)
 			)
 		)
@@
 		(dnp no)
 		(property "Reference" "TP705"
-			(at 113.03 114.84 0)
+			(at 113.03 116.11 0)
 			(do_not_autoplace yes)
 			(effects
@@
 			)
 		)
-		(property "Value" "TestPoint"
-			(at 113.03 116.75 0)
+		(property "Value" "REFP"
+			(at 113.03 112.44 0)
 			(do_not_autoplace yes)
 			(effects
@@
 				)
 				(justify left)
-				(hide yes)
 			)
 		)
@@
 			)
 		)
-		(property "Value" "TestPoint"
-			(at 113.03 126.83 0)
+		(property "Value" "REFN"
+			(at 113.03 127.32 0)
 			(do_not_autoplace yes)
 			(effects
@@
 				)
 				(justify right)
-				(hide yes)
 			)
 		)
@@
 		)
 		(property "Value" "GND"
-			(at 149.86 93.98 0)
+			(at 149.86 96.52 0)
 			(do_not_autoplace yes)
 			(effects
@@
 				)
 				(justify left)
-				(hide yes)
 			)
 		)
@@
 		)
 		(property "Value" "+5VA"
-			(at 218.44 38.1 0)
+			(at 215.9 33.02 0)
 			(do_not_autoplace yes)
 			(effects
@@
 					(size 1.27 1.27)
 				)
-				(justify left)
-				(hide yes)
 			)
 		)
@@
 		)
 		(property "Value" "GND"
-			(at 205.74 46.99 0)
+			(at 203.2 49.53 0)
 			(do_not_autoplace yes)
 			(effects
@@
 					(size 1.27 1.27)
 				)
-				(justify left)
-				(hide yes)
 			)
 		)
@@
 		)
 		(property "Value" "GND"
-			(at 215.9 46.99 0)
+			(at 213.36 49.53 0)
 			(do_not_autoplace yes)
 			(effects
@@
 					(size 1.27 1.27)
 				)
-				(justify left)
-				(hide yes)
 			)
 		)
@@
 		)
 		(property "Value" "+3V3"
-			(at 218.44 49.53 0)
+			(at 223.52 44.45 0)
 			(do_not_autoplace yes)
 			(effects
@@
 				)
 				(justify left)
-				(hide yes)
 			)
 		)
@@
 		)
 		(property "Value" "GND"
-			(at 205.74 58.42 0)
+			(at 203.2 60.96 0)
 			(do_not_autoplace yes)
 			(effects
@@
 					(size 1.27 1.27)
 				)
-				(justify left)
-				(hide yes)
 			)
 		)
@@
 		)
 		(property "Value" "GND"
-			(at 215.9 58.42 0)
+			(at 213.36 60.96 0)
 			(do_not_autoplace yes)
 			(effects
@@
 					(size 1.27 1.27)
 				)
-				(justify left)
-				(hide yes)
 			)
 		)
@@
 		)
 		(property "Value" "GND"
-			(at 185.42 91.44 0)
+			(at 177.8 93.98 0)
 			(do_not_autoplace yes)
 			(effects
@@
 					(size 1.27 1.27)
 				)
-				(justify left)
-				(hide yes)
+				(justify right)
 			)
 		)
@@
 			)
 		)
-		(property "Value" "TestPoint"
-			(at 212.09 104.4 0)
+		(property "Value" "DRDY"
+			(at 214.63 104.89 0)
 			(do_not_autoplace yes)
 			(effects
@@
 				)
 				(justify left)
-				(hide yes)
 			)
 		)
@@
 			)
 		)
-		(property "Value" "TestPoint"
-			(at 212.09 112.02 0)
+		(property "Value" "nCS"
+			(at 212.09 112.51 0)
 			(do_not_autoplace yes)
 			(effects
@@
 				)
 				(justify left)
-				(hide yes)
 			)
 		)
@@
 			)
 		)
-		(property "Value" "TestPoint"
-			(at 212.09 119.64 0)
+		(property "Value" "SCK"
+			(at 212.09 120.13 0)
 			(do_not_autoplace yes)
 			(effects
@@
 				)
 				(justify left)
-				(hide yes)
 			)
 		)
@@
 			)
 		)
-		(property "Value" "TestPoint"
-			(at 212.09 127.26 0)
+		(property "Value" "MOSI"
+			(at 212.09 127.75 0)
 			(do_not_autoplace yes)
 			(effects
@@
 				)
 				(justify left)
-				(hide yes)
 			)
 		)
@@
 			)
 		)
-		(property "Value" "TestPoint"
-			(at 212.09 134.88 0)
+		(property "Value" "MISO"
+			(at 212.09 135.37 0)
 			(do_not_autoplace yes)
 			(effects
@@
 				)
 				(justify left)
-				(hide yes)
 			)
 		)
@@
 			)
 		)
-		(property "Value" "TestPoint"
-			(at 203.2 96.78 0)
+		(property "Value" "GND"
+			(at 203.2 97.27 0)
 			(do_not_autoplace yes)
 			(effects
@@
 				)
 				(justify left)
-				(hide yes)
 			)
 		)
@@
 		)
 		(property "Value" "GND"
-			(at 214.63 105.41 0)
+			(at 212.09 107.95 0)
 			(do_not_autoplace yes)
 			(effects
@@
 					(size 1.27 1.27)
 				)
-				(justify left)
-				(hide yes)
 			)
 		)
@@
 			)
 		)
-		(property "Value" "TestPoint"
-			(at 203.2 142.5 0)
+		(property "Value" "GND"
+			(at 203.2 142.99 0)
 			(do_not_autoplace yes)
 			(effects
@@
 				)
 				(justify left)
-				(hide yes)
 			)
 		)
@@
 		)
 		(property "Value" "GND"
-			(at 214.63 151.13 0)
+			(at 212.09 153.67 0)
 			(do_not_autoplace yes)
 			(effects
@@
 					(size 1.27 1.27)
 				)
-				(justify left)
-				(hide yes)
 			)
 		)

Commit message: review r2 items 4-7: four per-sheet placement fixes
  4  linear_encoder - U601A's GND body ended at y=166.37 and U601E's +3V3 body
     began at exactly 166.37, so the two flags were touching. The whole U601E
     group drops 7.62 - unit, both flags, four wires, and the no_connect on its
     unused output, which does NOT ride with the symbol: ERC caught that as
     pin_not_connected plus a dangling no-connect the first time round.
  5  temp_sense - C704/C705's grounds sat 0.6 mm above the REFP row with
     TP705's reference on the row itself; the caps and grounds move up 5.08.
     Three verticals ran through the block title, so it is shortened to
     "CHANNEL 2 FILTER + SHARED REF", which at size 1.778 ends at x=135.9 and
     clears the leftmost of them at 137.16.
  6  ui_io - R915's reference sat on its own body. It is the horizontal 0R
     variant but its fields were still on the vertical pattern; moved to the
     _H symbol's own pattern.
  7  motor_drive - #PWR1109/#PWR1110 bodies ended exactly on the block border
     and their GND text was outside the box entirely. Both move up to 138.43.

ERC 0 errors / 0 warnings at severity-all; 412 components, 259 nets, node sets
identical - all four are placement only.

Co-Authored-By: Claude Opus 5 <noreply@anthropic.com>
Claude-Session: https://claude.ai/code/session_01PFWfwT8RZc8Zqn8vgZxV8j
Other:
- note added: "CHANNEL 2 FILTER + SHARED REF"
- note removed: "CHANNEL 2 FILTER AND SHARED REFERENCE"
- moved on the sheet: C704, C705
Changed lines of the file:
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@@
 		(comment 4 "Reasoning + root-sheet needs: docs/decisions/actuator-sch-afe.md")
 	)
+	(wire
+		(pts
+			(xy 109.22 91.44) (xy 109.22 101.6)
+		)
+		(stroke
+			(width 0)
+			(type default)
+		)
+	)
+	(wire
+		(pts
+			(xy 119.38 96.52) (xy 119.38 101.6)
+		)
+		(stroke
+			(width 0)
+			(type default)
+		)
+	)
 	(symbol
 		(lib_id "Amodo_Connectors:1752120")
@@
 	(symbol
 		(lib_id "Amodo_Capacitors:CAP_MLCC_10nF_0603_5%_100V")
-		(at 109.22 109.22 0)
+		(at 109.22 104.14 0)
 		(unit 1)
 		(exclude_from_sim no)
@@
 		(dnp no)
 		(property "Reference" "C704"
-			(at 111.51 108.58 0)
+			(at 111.51 103.5 0)
 			(do_not_autoplace yes)
 			(effects
@@
 		)
 		(property "Value" "10nF"
-			(at 111.51 110.49 0)
+			(at 111.51 105.41 0)
 			(do_not_autoplace yes)
 			(effects
@@
 		)
 		(property "Footprint" "Amodo:C_0603_1608Metric"
-			(at 109.22 109.22 0)
+			(at 109.22 104.14 0)
 			(do_not_autoplace yes)
 			(effects
@@
 		)
 		(property "Datasheet" "https://product.tdk.com/system/files/dam/doc/product/capacitor/ceramic/mlcc/catalog/mlcc_automotive_esd_en.pdf"
-			(at 109.22 109.22 0)
+			(at 109.22 104.14 0)
 			(do_not_autoplace yes)
 			(effects
@@
 		)
 		(property "Description" "SMD MLCC Capacitor 10nF 0603 5% C0G 100V"
-			(at 109.22 109.22 0)
+			(at 109.22 104.14 0)
 			(do_not_autoplace yes)
 			(effects
@@
 		)
 		(property "mpn" "CGA3EAC0G2A103J080AC"
-			(at 109.22 109.22 0)
+			(at 109.22 104.14 0)
 			(do_not_autoplace yes)
 			(effects
@@
 		)
 		(property "SymLifecycle" "reviewed"
-			(at 109.22 109.22 0)
+			(at 109.22 104.14 0)
 			(do_not_autoplace yes)
 			(effects
@@
 	(symbol
 		(lib_id "Amodo_Symbols:GND")
-		(at 109.22 111.76 0)
+		(at 109.22 106.68 0)
 		(unit 1)
 		(exclude_from_sim no)
@@
 		(dnp no)
 		(property "Reference" "#PWR706"
-			(at 111.76 110.49 0)
+			(at 109.22 106.68 0)
 			(do_not_autoplace yes)
 			(effects
@@
 		)
 		(property "Value" "GND"
-			(at 109.22 115.57 0)
+			(at 109.22 110.49 0)
 			(do_not_autoplace yes)
 			(effects
@@
 		)
 		(property "Footprint" ""
-			(at 109.22 111.76 0)
+			(at 109.22 106.68 0)
 			(do_not_autoplace yes)
 			(effects
@@
 		)
 		(property "Datasheet" ""
-			(at 109.22 111.76 0)
+			(at 109.22 106.68 0)
 			(do_not_autoplace yes)
 			(effects
@@
 		)
 		(property "Description" "Power symbol creates a global label with name \"GND\" , ground"
-			(at 109.22 111.76 0)
+			(at 109.22 106.68 0)
 			(do_not_autoplace yes)
 			(effects
@@
 		)
 		(property "SymLifecycle" "tested"
-			(at 109.22 111.76 0)
+			(at 109.22 106.68 0)
 			(do_not_autoplace yes)
 			(effects
@@
 	(symbol
 		(lib_id "Amodo_Capacitors:CAP_MLCC_10nF_0603_5%_100V")
-		(at 119.38 109.22 0)
+		(at 119.38 104.14 0)
 		(unit 1)
 		(exclude_from_sim no)
@@
 		(dnp no)
 		(property "Reference" "C705"
-			(at 121.67 108.58 0)
+			(at 121.67 103.5 0)
 			(do_not_autoplace yes)
 			(effects
@@
 		)
 		(property "Value" "10nF"
-			(at 121.67 110.49 0)
+			(at 121.67 105.41 0)
 			(do_not_autoplace yes)
 			(effects
@@
 		)
 		(property "Footprint" "Amodo:C_0603_1608Metric"
-			(at 119.38 109.22 0)
+			(at 119.38 104.14 0)
 			(do_not_autoplace yes)
 			(effects
@@
 		)
 		(property "Datasheet" "https://product.tdk.com/system/files/dam/doc/product/capacitor/ceramic/mlcc/catalog/mlcc_automotive_esd_en.pdf"
-			(at 119.38 109.22 0)
+			(at 119.38 104.14 0)
 			(do_not_autoplace yes)
 			(effects
@@
 		)
 		(property "Description" "SMD MLCC Capacitor 10nF 0603 5% C0G 100V"
-			(at 119.38 109.22 0)
+			(at 119.38 104.14 0)
 			(do_not_autoplace yes)
 			(effects
@@
 		)
 		(property "mpn" "CGA3EAC0G2A103J080AC"
-			(at 119.38 109.22 0)
+			(at 119.38 104.14 0)
 			(do_not_autoplace yes)
 			(effects
@@
 		)
 		(property "SymLifecycle" "reviewed"
-			(at 119.38 109.22 0)
+			(at 119.38 104.14 0)
 			(do_not_autoplace yes)
 			(effects
@@
 	(symbol
 		(lib_id "Amodo_Symbols:GND")
-		(at 119.38 111.76 0)
+		(at 119.38 106.68 0)
 		(unit 1)
 		(exclude_from_sim no)
@@
 		(dnp no)
 		(property "Reference" "#PWR707"
-			(at 121.92 110.49 0)
+			(at 119.38 106.68 0)
 			(do_not_autoplace yes)
 			(effects
@@
 		)
 		(property "Value" "GND"
-			(at 121.92 115.57 0)
+			(at 119.38 110.49 0)
 			(do_not_autoplace yes)
 			(effects
@@
 		)
 		(property "Footprint" ""
-			(at 119.38 111.76 0)
+			(at 119.38 106.68 0)
 			(do_not_autoplace yes)
 			(effects
@@
 		)
 		(property "Datasheet" ""
-			(at 119.38 111.76 0)
+			(at 119.38 106.68 0)
 			(do_not_autoplace yes)
 			(effects
@@
 		)
 		(property "Description" "Power symbol creates a global label with name \"GND\" , ground"
-			(at 119.38 111.76 0)
+			(at 119.38 106.68 0)
 			(do_not_autoplace yes)
 			(effects
@@
 		)
 		(property "SymLifecycle" "tested"
-			(at 119.38 111.76 0)
+			(at 119.38 106.68 0)
 			(do_not_autoplace yes)
 			(effects
@@
 	)
 	(text
-		"CHANNEL 2 FILTER AND SHARED REFERENCE"
+		"CHANNEL 2 FILTER + SHARED REF"
 		(exclude_from_sim no)
 		(at 87.63 79.76 0)
@@
 		)
 		(stroke
-			(width 0)
-			(type default)
-		)
-	)
-	(wire
-		(pts
-			(xy 109.22 91.44) (xy 109.22 106.68)
-		)
-		(stroke
-			(width 0)
-			(type default)
-		)
-	)
-	(wire
-		(pts
-			(xy 119.38 96.52) (xy 119.38 106.68)
-		)
-		(stroke
