File: hardware/kicad/faff2_cbs1/temp_sense.kicad_sch (KiCad schematic)
At the start: 44 parts, among them J701 1752120, J702 1752120, U701 ADS1120

Commit message: review r2 item 8: one placement rule for every power symbol's net name
"Directly above it, centre justified, and close" - applied as no sideways
offset, centred, 3.81 mm away: above a rail arrow, below a ground. All 283
power symbols now carry it; 103 did not, most left-anchored rather than centred
and a few offset up to 7.6 mm sideways by round 1's auto-placer.

The ground mirror is an interpretation and is flagged as such: "above" a GND
symbol is where its wire arrives, and 137 instances plus every convention put
GND's name under the triangle. One line to change if the captain meant it
literally.

What makes this different from round 1 is that the label is now PINNED, so
everything else moves instead - the symbol along its own stub, a note to the
nearest clear spot, a block box outward (five rectangles grew where a name sat
on a border with clear space beyond), and two PWR_FLAGs placed by hand because
their 9.5 mm names do not fit the 10 mm rail runs they tap.

Thirteen of 283 still graze a wire, body or note on the two densest sheets and
are listed in the decisions file rather than hidden. Each needs the parts around
it respaced, which is more than a label sweep should do unasked - the TIM1 note
on motor_drive in particular has nowhere to go: no clear position exists for a
47.6 x 8.7 mm box anywhere in that block.

Also recorded: my own severity metric scored wire-through-text at zero for a
while, because a wire is a zero-thickness segment and box-intersection depth
against it is always 0. For those, severity is how far inside the box the line
sits. A render caught it; the number did not.

ERC 0 errors / 0 warnings at severity-all; 412 components, 259 nets, node sets
identical to before the batch. Review PDF regenerated once, here, for the whole
of round 2.

Co-Authored-By: Claude Opus 5 <noreply@anthropic.com>
Claude-Session: https://claude.ai/code/session_01PFWfwT8RZc8Zqn8vgZxV8j
Changed lines of the file:
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@@
 		)
 		(property "Value" "GND"
-			(at 71.12 48.26 0)
+			(at 71.12 46.99 0)
 			(do_not_autoplace yes)
 			(effects
@@
 		)
 		(property "Value" "GND"
-			(at 71.12 116.84 0)
+			(at 71.12 115.57 0)
 			(do_not_autoplace yes)
 			(effects
@@
 					(size 1.27 1.27)
 				)
-				(justify left)
 			)
 		)
@@
 		)
 		(property "Value" "GND"
-			(at 109.22 143.51 0)
+			(at 109.22 138.43 0)
 			(do_not_autoplace yes)
 			(effects
@@
 		)
 		(property "Value" "GND"
-			(at 119.38 143.51 0)
+			(at 119.38 138.43 0)
 			(do_not_autoplace yes)
 			(effects
@@
 		)
 		(property "Value" "GND"
-			(at 149.86 96.52 0)
+			(at 147.32 96.52 0)
 			(do_not_autoplace yes)
 			(effects
@@
 					(size 1.27 1.27)
 				)
-				(justify left)
 			)
 		)
@@
 		)
 		(property "Value" "100nF"
-			(at 215.65 44.45 0)
+			(at 216.92 45.72 0)
 			(do_not_autoplace yes)
 			(effects
@@
 		)
 		(property "Value" "+3V3"
-			(at 223.52 44.45 0)
+			(at 215.9 44.45 0)
 			(do_not_autoplace yes)
 			(effects
@@
 					(size 1.27 1.27)
 				)
-				(justify left)
 			)
 		)
@@
 		)
 		(property "Value" "GND"
-			(at 177.8 93.98 0)
+			(at 182.88 93.98 0)
 			(do_not_autoplace yes)
 			(effects
@@
 					(size 1.27 1.27)
 				)
-				(justify right)
 			)
 		)
@@
 	(rectangle
 		(start 17.78 11.43)
-		(end 84.46 46.99)
+		(end 84.46 49.53)
 		(stroke
 			(width 0.1524)
@@
 	(rectangle
 		(start 17.78 78.74)
-		(end 84.46 115.57)
+		(end 84.46 118.11)
 		(stroke
 			(width 0.1524)
@@
 	(rectangle
 		(start 86.36 78.74)
-		(end 146.05 146.05)
+		(end 149.86 146.05)
 		(stroke
 			(width 0.1524)
@@
 		"R707 is the shared reference resistor -\nboth return leads meet here, so both\nchannels are ratiometric."
 		(exclude_from_sim no)
-		(at 96.52 137.16 0)
+		(at 96.52 139.7 0)
 		(effects
 			(font
@@
 		"ADS1120 SUPPLIES AND SPI2"
 		(exclude_from_sim no)
-		(at 181.61 32.77 0)
+		(at 181.61 28.96 0)
 		(effects
 			(font
