File: hardware/kicad/faff2_cbs1/power_entry_24v.kicad_sch (KiCad schematic)
At the start: 28 parts, among them J201 KPJX-4S, Q201 DMP6023LFG-7

Commit message: review r3 item 4: respace every grazing placement, and rehome the TIM1 note
Round 2 left thirteen power-symbol names grazing something and pinned the
labels. Item 1's checker turned thirteen into sixty once labels and bodies
became subjects and the font model learned that block titles are bold 1.778 -
40% wider per character than the 1.27 it had assumed, which is how a 35 mm
title came back as 25. Fifty-seven are now clear. ERC 0/0 and node sets
identical: every change here is geometry.

The dominant defect, ten times over, is a power symbol's arrow with a vertex
exactly on a wire that runs past it and does not connect - the same thing the
captain screenshotted, nine more times. Each moves along its own stub: GND
arrows up, rail arrows down, because a rail arrow's name sits above it and
moving up only puts the text where the arrow was.

The rest: six bold titles wider than their block, eight notes and labels running
out through a border, twelve pinned names overlapped by a neighbour that moved
instead, and both 5 V PWR_FLAGs, which move onto the test-point stub below where
their 9.5 mm name has clear air.

Two checker corrections came out of doing the work. Fourteen findings were text
over its OWN conductor - a label on its wire with a branch of the same net
dropping through the text, which is what "the wire must extend under the entire
label" asks for; wire_nodes() groups segments into electrical nodes and excuses
the whole node. And field-against-field comparison had been lost in the
subject/obstacle rewrite - reference-against-value is the commonest defect there
is, and it went unnoticed until a render showed PWR_FLAG 0.86 mm inside a
neighbouring 100nF on a sheet the checker called clean.

The TIM1 note: round 2 recorded that nothing 47.6 x 8.7 fitted anywhere in
motor_drive block 4. With item 1's geometry that was wrong - 495 positions fit.
It now sits beside U1101's logic inputs, which is what it describes.

Three are left, both explained in the decisions file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
Changed lines of the file:
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@@
 	(wire
 		(pts
-			(xy 71.12 45.72) (xy 81.28 45.72)
+			(xy 71.12 45.72) (xy 77.47 45.72)
 		)
 		(stroke
@@
 	(symbol
 		(lib_id "Amodo_Symbols:PWR_FLAG")
-		(at 81.28 45.72 0)
+		(at 77.47 45.72 0)
 		(unit 1)
 		(exclude_from_sim no)
@@
 		(fields_autoplaced no)
 		(property "Reference" "#FLG203"
-			(at 83.82 44.45 0)
+			(at 80.01 44.45 0)
 			(effects
 				(font
@@
 		)
 		(property "Value" "PWR_FLAG"
-			(at 81.28 41.91 0)
+			(at 77.47 41.91 0)
 			(effects
 				(font
@@
 		)
 		(property "Footprint" ""
-			(at 81.28 45.72 0)
+			(at 77.47 45.72 0)
 			(effects
 				(font
@@
 		)
 		(property "Datasheet" ""
-			(at 81.28 45.72 0)
+			(at 77.47 45.72 0)
 			(effects
 				(font
@@
 		)
 		(property "Description" "Special symbol for telling ERC where power comes from"
-			(at 81.28 45.72 0)
+			(at 77.47 45.72 0)
 			(effects
 				(font
@@
 		)
 		(property "SymLifecycle" "tested"
-			(at 81.28 45.72 0)
+			(at 77.47 45.72 0)
 			(effects
 				(font
@@
 		)
 		(property "ki_keywords" "flag power"
-			(at 81.28 45.72 0)
-			(effects
-				(font
+			(at 77.47 45.72 0)
+			(effects
+				(font
