File: hardware/kicad/faff2_cbs1/loadcell_afe.kicad_sch (KiCad schematic)
At the start: 52 parts, among them J501 1729076, J502 8510-4500PL, U501 ADS1235

Commit message: review r3 item 4: respace every grazing placement, and rehome the TIM1 note
Round 2 left thirteen power-symbol names grazing something and pinned the
labels. Item 1's checker turned thirteen into sixty once labels and bodies
became subjects and the font model learned that block titles are bold 1.778 -
40% wider per character than the 1.27 it had assumed, which is how a 35 mm
title came back as 25. Fifty-seven are now clear. ERC 0/0 and node sets
identical: every change here is geometry.

The dominant defect, ten times over, is a power symbol's arrow with a vertex
exactly on a wire that runs past it and does not connect - the same thing the
captain screenshotted, nine more times. Each moves along its own stub: GND
arrows up, rail arrows down, because a rail arrow's name sits above it and
moving up only puts the text where the arrow was.

The rest: six bold titles wider than their block, eight notes and labels running
out through a border, twelve pinned names overlapped by a neighbour that moved
instead, and both 5 V PWR_FLAGs, which move onto the test-point stub below where
their 9.5 mm name has clear air.

Two checker corrections came out of doing the work. Fourteen findings were text
over its OWN conductor - a label on its wire with a branch of the same net
dropping through the text, which is what "the wire must extend under the entire
label" asks for; wire_nodes() groups segments into electrical nodes and excuses
the whole node. And field-against-field comparison had been lost in the
subject/obstacle rewrite - reference-against-value is the commonest defect there
is, and it went unnoticed until a render showed PWR_FLAG 0.86 mm inside a
neighbouring 100nF on a sheet the checker called clean.

The TIM1 note: round 2 recorded that nothing 47.6 x 8.7 fitted anywhere in
motor_drive block 4. With item 1's geometry that was wrong - 495 positions fit.
It now sits beside U1101's logic inputs, which is what it describes.

Three are left, both explained in the decisions file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
Changed lines of the file:
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@@
 		"SIGNAL INPUT FILTER"
 		(exclude_from_sim no)
-		(at 96.52 41.66 0)
+		(at 100.33 41.66 0)
 		(effects
 			(font
@@
 		"REFERENCE (SENSE) FILTER - RATIOMETRIC"
 		(exclude_from_sim no)
-		(at 96.52 84.84 0)
+		(at 100.33 84.84 0)
 		(effects
 			(font
@@
 	)
 	(rectangle
-		(start 196.85 13.97)
-		(end 245.11 35.56)
+		(start 196.85 16.51)
+		(end 254 35.56)
 		(stroke
 			(width 0.1524)
@@
 		"5 V BRIDGE EXCITATION"
 		(exclude_from_sim no)
-		(at 198.12 14.99 0)
+		(at 216.51 17.15 0)
 		(effects
 			(font
@@
 		"OPERATING POINT (prelim calc Force sheet; ADS1235 SBAS824)\n  Gain 128, 4800 SPS, Sinc2, VREF = bridge excitation (ratiometric)\n  FSR = +/-VREF/128 = +/-39.06 mV (78.125 mV span) vs +/-10 mV signal\n  Input-referred noise 0.29 uVrms / 2.4 uVpp (data sheet table 1)\n    = 12.0 mNpp (V50N) / 2.4 mNpp (V10N) vs REQ-FF-04 20 / 5 mNpp\n  Ratiometric operation cancels excitation drift and noise, so the\n  5 V rail does not need to be a precision reference.\n\nFILTERS - the ADS1235 data sheet figure 84 reference design.\n  Signal and reference filters are deliberately identical so their\n  corner frequencies match: 100R series per leg, 1 nF C0G common mode\n  to AVSS, 10 nF C0G differential. The differential capacitor is 10x\n  the common-mode capacitors, so common-mode capacitor mismatch\n  converts little common-mode noise into differential noise.\n  Differential corner ~76 kHz, common mode ~1.6 MHz; the ADC PGA\n  antialias filter (C514, 4.7 nF C0G) is at 60 kHz.\n  R505 (100k) across the sense pair is the data sheet reference\n  monitor resistor: it collapses VREF if the cable is unplugged so\n  REFL_ALM asserts. It sits on the bridge side of R503/R504 so its\n  50 uA does not develop an error across the reference filter."
 		(exclude_from_sim no)
-		(at 250.19 76.2 0)
+		(at 251.46 76.2 0)
 		(effects
 			(font

Commit message: review r4 items 2,3,5,6,9: PGND, the frame boundary, and the U.FL connectors
Item 2, U304's PGND ground sitting on top of C318: the answer was already on
the sheet. U301 is the same regulator wired the same way, and its PGND ground
hangs 1.27 mm below the pin with its name clear above the VCC stub; U304's hung
6.35 mm down, which put it in C318's lane. Making it match U301 also closes both
of round 3's residual findings - power_rails is clear for the first time.

Item 3, the +5VA symbol outside the sheet boundary: the drawing area starts at
y=11.94, measured off a render, and the "+5VA" name's box ran 10.79..12.06 -
straddling it, inside the frame's ruler band. The whole excitation cluster drops
6.35 mm, the block box follows, and the feed keeps its long run and doglegs down
to the new row.

Item 9 is the same defect: temp_sense's PROBE 1 and CHANNEL 1 FILTER rectangles
start at y=11.43, half a millimetre above the drawing area. So do four of mcu's,
laid out to the same wrong value, so both sheets are fixed - every top edge to
12.70 and the titles under them to 13.34. Nothing on any sheet is above the
boundary now.

Item 5, FL501/FL502 -> J503/J504. The captain is right and there is no reason
that survives: they are Amodo_Connectors:CONUFL001-SMD, U.FL coaxial
connectors, with connector footprints, and the library symbol's own default
reference prefix is J. The FL prefix was an instance-level override
contradicting the part, and in IEEE-315 FL designates a filter. They sit in a
filter chain, which is the only reading that explains it. DEC-A14 records it.

Item 6, a concise pin-out beside J501. The full table was in the notes column
90 mm away; this is the five-line version directly under the connector, where
somebody landing a cable will look. Width is capped by the signal wires
dropping at x=48.26.

ERC 0/0 at severity-all; 408 components, 264 nets. The only netlist change is
item 5's re-designation - same nets, same members, new names.

Co-Authored-By: Claude Opus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
Parts:
- renumbered FL501 to J503, FL502 to J504
Other:
- note added: "J501 -> HBK S2M cable 1 SIG+ wht 2 SIG- red 3 EXC+ blu 4 SEN+ grn 5 SEN- gry 6 EXC- blk 7,8 SHLD screen, R510"
- note added: "TEST AND ISOLATION PROVISIONS (TEST_PLAN.md section 4) TP501 excitation+ TP502/TP503 sense+/- TP504/TP505 ADC reference J503/J504 U.FL on the ADC-side SIG+/SIG- nodes - the noise-floor measurement that decides REQ-FF-04. Placed symmetrically so the differential pair stays balanced (TEST_PLAN section 2.3). J502 logic-analyser header (Amodo keyed 0.1in socket, 8510-4500PL) carries the whole digital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"
- note removed: "TEST AND ISOLATION PROVISIONS (TEST_PLAN.md section 4) TP501 excitation+ TP502/TP503 sense+/- TP504/TP505 ADC reference FL501/FL502 U.FL on the ADC-side SIG+/SIG- nodes - the noise-floor measurement that decides REQ-FF-04. Placed symmetrically so the differential pair stays balanced (TEST_PLAN section 2.3). J502 logic-analyser header (Amodo keyed 0.1in socket, 8510-4500PL) carries the whole digit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"
- moved on the sheet: C507, C508, R508
