File: hardware/kicad/faff2_cbs1/mcu.kicad_sch (KiCad schematic)
At the start: 62 parts, among them J1001 USB_C_Receptacle_USB2.0_16P, J1002 TSW-105-07-F-D, J1003 TSW-105-07-F-D, J1004 PH1-06-UA, SW1001 PTS526, U1001 STM32H723VET6, U1002 USB3320C, U1003 SRAM 32Mb, U1004 MIC5365-1.8, Y1001 24MHz, Y1002 24MHz 18pF

Commit message: review r3 item 4: respace every grazing placement, and rehome the TIM1 note
Round 2 left thirteen power-symbol names grazing something and pinned the
labels. Item 1's checker turned thirteen into sixty once labels and bodies
became subjects and the font model learned that block titles are bold 1.778 -
40% wider per character than the 1.27 it had assumed, which is how a 35 mm
title came back as 25. Fifty-seven are now clear. ERC 0/0 and node sets
identical: every change here is geometry.

The dominant defect, ten times over, is a power symbol's arrow with a vertex
exactly on a wire that runs past it and does not connect - the same thing the
captain screenshotted, nine more times. Each moves along its own stub: GND
arrows up, rail arrows down, because a rail arrow's name sits above it and
moving up only puts the text where the arrow was.

The rest: six bold titles wider than their block, eight notes and labels running
out through a border, twelve pinned names overlapped by a neighbour that moved
instead, and both 5 V PWR_FLAGs, which move onto the test-point stub below where
their 9.5 mm name has clear air.

Two checker corrections came out of doing the work. Fourteen findings were text
over its OWN conductor - a label on its wire with a branch of the same net
dropping through the text, which is what "the wire must extend under the entire
label" asks for; wire_nodes() groups segments into electrical nodes and excuses
the whole node. And field-against-field comparison had been lost in the
subject/obstacle rewrite - reference-against-value is the commonest defect there
is, and it went unnoticed until a render showed PWR_FLAG 0.86 mm inside a
neighbouring 100nF on a sheet the checker called clean.

The TIM1 note: round 2 recorded that nothing 47.6 x 8.7 fitted anywhere in
motor_drive block 4. With item 1's geometry that was wrong - 495 positions fit.
It now sits beside U1101's logic inputs, which is what it describes.

Three are left, both explained in the decisions file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
Other:
- note added: "D OCTOSPI1 FORCE-PROFILE RAM (QPI PSRAM) REQ-AR-12"
- note removed: "D OCTOSPI1 FORCE-PROFILE RAM (QPI PSRAM) REQ-AR-12 / DEC-0006"
Changed lines of the file:
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@@
 		(fill (type none))
 	)
-	(text "D  OCTOSPI1 FORCE-PROFILE RAM (QPI PSRAM)  REQ-AR-12 / DEC-0006"
+	(text "D  OCTOSPI1 FORCE-PROFILE RAM (QPI PSRAM)  REQ-AR-12"
 		(exclude_from_sim no)
 		(at 105.41 83.82 0)
@@
 		)
 	)
-	(text "USB 2.0 data only: no VBUS load, no sink, no PD (REQ-EL-10, DEC-0002).\n5.1k Rd on both CC lines is what makes this a valid USB-C device attachment.\nVBUS is SENSED ONLY, through RVBUS in block F, so the PHY SessVld comparator\ntells firmware a host is present - which is why VBUS_MON (PC5) stays free for\nthe motor DC link (supports OQ-01 / DEC-0011). CC carries nothing but the two\nRd resistors, so it needs no ESD part; the high-speed pair has the USBLC6-2P6."
+	(text "USB 2.0 data only: no VBUS load, no sink, no PD (REQ-EL-10, DEC-0002).\n5.1k Rd on both CC lines is what makes this a valid USB-C device\nattachment. VBUS is SENSED ONLY, through RVBUS in block F, so the PHY\nSessVld comparator tells firmware a host is present - which is why\nVBUS_MON (PC5) stays free for the motor DC link (supports OQ-01 /\nDEC-0011). CC carries nothing but the two Rd resistors, so it needs no\nESD part; the high-speed pair has the USBLC6-2P6."
 		(exclude_from_sim no)
-		(at 322.58 66.04 0)
+		(at 316.23 66.04 0)
 		(effects (font (size 1.27 1.27)) (justify left top))
 	)
@@
 	(hierarchical_label "LINEAR_ENCODER_A"
 		(shape input)
-		(at 43.18 161.29 0)
+		(at 45.72 161.29 0)
 		(effects (font (size 1.27 1.27)) (justify right bottom))
 	)
 	(hierarchical_label "LINEAR_ENCODER_B"
 		(shape input)
-		(at 43.18 163.83 0)
+		(at 45.72 163.83 0)
 		(effects (font (size 1.27 1.27)) (justify right bottom))
 	)
 	(hierarchical_label "LINEAR_ENCODER_Z"
 		(shape input)
-		(at 43.18 166.37 0)
+		(at 45.72 166.37 0)
 		(effects (font (size 1.27 1.27)) (justify right bottom))
 	)
@@
 		(stroke (width 0) (type default))
 	)
-	(wire (pts (xy 43.18 161.29) (xy 63.5 161.29))
+	(wire (pts (xy 45.72 161.29) (xy 63.5 161.29))
 		(stroke (width 0) (type default))
 	)
-	(wire (pts (xy 43.18 163.83) (xy 63.5 163.83))
+	(wire (pts (xy 45.72 163.83) (xy 63.5 163.83))
 		(stroke (width 0) (type default))
 	)
-	(wire (pts (xy 43.18 166.37) (xy 63.5 166.37))
+	(wire (pts (xy 45.72 166.37) (xy 63.5 166.37))
 		(stroke (width 0) (type default))
 	)

Commit message: review r4 items 2,3,5,6,9: PGND, the frame boundary, and the U.FL connectors
Item 2, U304's PGND ground sitting on top of C318: the answer was already on
the sheet. U301 is the same regulator wired the same way, and its PGND ground
hangs 1.27 mm below the pin with its name clear above the VCC stub; U304's hung
6.35 mm down, which put it in C318's lane. Making it match U301 also closes both
of round 3's residual findings - power_rails is clear for the first time.

Item 3, the +5VA symbol outside the sheet boundary: the drawing area starts at
y=11.94, measured off a render, and the "+5VA" name's box ran 10.79..12.06 -
straddling it, inside the frame's ruler band. The whole excitation cluster drops
6.35 mm, the block box follows, and the feed keeps its long run and doglegs down
to the new row.

Item 9 is the same defect: temp_sense's PROBE 1 and CHANNEL 1 FILTER rectangles
start at y=11.43, half a millimetre above the drawing area. So do four of mcu's,
laid out to the same wrong value, so both sheets are fixed - every top edge to
12.70 and the titles under them to 13.34. Nothing on any sheet is above the
boundary now.

Item 5, FL501/FL502 -> J503/J504. The captain is right and there is no reason
that survives: they are Amodo_Connectors:CONUFL001-SMD, U.FL coaxial
connectors, with connector footprints, and the library symbol's own default
reference prefix is J. The FL prefix was an instance-level override
contradicting the part, and in IEEE-315 FL designates a filter. They sit in a
filter chain, which is the only reading that explains it. DEC-A14 records it.

Item 6, a concise pin-out beside J501. The full table was in the notes column
90 mm away; this is the five-line version directly under the connector, where
somebody landing a cable will look. Width is capped by the signal wires
dropping at x=48.26.

ERC 0/0 at severity-all; 408 components, 264 nets. The only netlist change is
item 5's re-designation - same nets, same members, new names.

Co-Authored-By: Claude Opus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
Changed lines of the file:
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@@
 		(comment 4 "Reasoning: docs/decisions/actuator-sch-mcu.md")
 	)
-	(rectangle (start 22.86 11.43) (end 198.12 78.74)
+	(rectangle (start 22.86 12.7) (end 198.12 78.74)
 		(stroke (width 0.2) (type solid))
 		(fill (type none))
@@
 	(text "A  MCU CORE - SUPPLIES, RESET, BOOT, HSE CLOCK IN"
 		(exclude_from_sim no)
-		(at 24.13 12.7 0)
+		(at 24.13 13.34 0)
 		(effects (font (size 1.6 1.6) (bold yes)) (justify left top))
 	)
@@
 		(effects (font (size 1.27 1.27)) (justify left top))
 	)
-	(rectangle (start 202.31 11.43) (end 295.91 139.7)
+	(rectangle (start 202.31 12.7) (end 295.91 139.7)
 		(stroke (width 0.2) (type solid))
 		(fill (type none))
@@
 	(text "F  USB3320C Hi-SPEED ULPI PHY  (REQ-AR-13)"
 		(exclude_from_sim no)
-		(at 203.58 12.7 0)
+		(at 203.58 13.34 0)
 		(effects (font (size 1.6 1.6) (bold yes)) (justify left top))
 	)
@@
 		(effects (font (size 1.27 1.27)) (justify left top))
 	)
-	(rectangle (start 297.18 11.43) (end 407.67 80.01)
+	(rectangle (start 297.18 12.7) (end 407.67 80.01)
 		(stroke (width 0.2) (type solid))
 		(fill (type none))
@@
 	(text "G  USB-C RECEPTACLE - DATA ONLY, NO BUS POWER, NO PD"
 		(exclude_from_sim no)
-		(at 298.45 12.7 0)
+		(at 298.45 13.34 0)
 		(effects (font (size 1.6 1.6) (bold yes)) (justify left top))
 	)
@@
 	)
 	(rectangle
-		(start 411.48 11.43)
+		(start 411.48 12.7)
 		(end 581.66 88.9)
 		(stroke
@@
 	(text "C  USB3320 24 MHz CRYSTAL  (ITS OWN REFERENCE)"
 		(exclude_from_sim no)
-		(at 412.75 12.7 0)
+		(at 412.75 13.34 0)
 		(effects
 			(font

Commit message: review r4 items 10,11: the SWD header becomes the STM32 14-way part
J1003 was a 2x5 2.54 mm header on the ARM Cortex Debug 10-pin order. It is now
Amodo_Connectors:SAMTEC_SHF-107-01-L-D-SM, the 14-way 1.27 mm IDC socket
ARIA_EITSYS_CBs_1 uses for the same job - a house-library part, so nothing goes
project-local. The pinout is copied from that repo's Microcontroller.kicad_sch,
J11, traced pin by pin from a read-only sparse clone rather than assumed:
1/2 NC, 3 VDD through 100R, 4 SWDIO, 5 GND, 6 SWCLK, 7 GND, 8/9/10 NC, 11 GND,
12 nRESET, 13 UART RX, 14 UART TX.

ONE deviation, and it is an addition: SWO goes on pin 10, which is NC there.
This design has SWO (REQ-AR-15) and the reference board does not; dropping it to
match exactly would remove a capability, and pin 10 is a spare in the signal
column, so a cable wired for that board just leaves it open. Flagged in the
sheet note and for the captain.

Item 10's 100R between the header and +3V3 is R1015 - the same series resistance
their R625 puts on the same pin, which is why the two items arrived together.
R1013 and R1014 already existed on DBG_RX and DBG_TX and keep their jobs; all
three are horizontal now, on the house symbol rotated 90 with field angles
compensated. The three separate GND flags become one rail with a single flag,
which is schematic-style's rule for a 2.54 mm pin row.

Two tooling bugs fixed on the way, both of which had been quietly wrong for
several commits. Labels were being addressed by an occurrence index, and every
one of these nets is labelled at BOTH ends - so "the first SWDIO" was the one at
the MCU pin, and moving it left four labels dangling. They are keyed by position
now. And sch_edit.add() inserted one tab too many in front of everything it
added: KiCad does not care, but every tool here that anchors on a line start
stopped seeing those blocks, so a resistor that was in the netlist could not be
found on the sheet. Every round-4 script was re-run after the fix.

ERC 0/0 at severity-all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
Parts:
- removed J1003: TSW-105-07-F-D, Amodo:TSW-105-07-F-D, symbol Amodo_Connectors:Header_Male_10-way_2-row_Straight_2.54mm_THT
- added J1003: SAMTEC_SHF-107-01-L-D-SM, Amodo:SAMTEC_SHF-107-01-L-D-SM, symbol Amodo_Connectors:SAMTEC_SHF-107-01-L-D-SM
- added R1015: 100R, Amodo:R_0603_1608Metric, symbol Amodo_Resistors:RES_TF_100R_0603
Connections:
- net +3V3: now also R1015.1
- net DBG_RX: now also R1013.1; no longer R1013.2
- net GND: now also J1003.11, J1003.5, J1003.7
- net MCU_nRESET: now also J1003.12
- net SWCLK: now also J1003.6
- net SWDIO: now also J1003.4
- net SWO: now also J1003.10
- net at R1014.1: now also J1003.14
- new net: J1003.13, R1013.2
- new net: J1003.3, R1015.2
- no-connect marks 10 -> 14
Other:
- note added: "PINOUT - the STM32 14-way 1.27 mm IDC order, copied pin for pin from ARIA_EITSYS_CBs_1 (Microcontroller.kicad_sch, J11) so one debug cable serves both boards: 1 NC 2 NC 3 VDD (+3V3 via R1015 100R) 4 SWDIO 5 GND 6 SWCLK 7 GND 8 NC 9 NC 10 SWO 11 GND 12 nRESET 13 DBG_RX 14 DBG_TX SWO on pin 10 is this board's ONE addition: pin 10 is NC on the reference board, this design has SWO (REQ-AR-15), and a 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"
- note removed: "PINOUT - standard ARM Cortex Debug 10-pin order on 2.54 mm pitch, so a 2x5 SWD probe cable plugs straight on: 1 VTref (+3V3) 2 SWDIO 3 GND 4 SWCLK 5 GND 6 SWO 7 DBG_RX 8 DBG_TX 9 GND 10 nRESET Pins 7 and 8 are KEY / NC on the ARM pinout and are reused here for the USART3 console (REQ-AR-15 and the block diagram both put SWD and UART on ONE header). They are SWD-safe: an SWD probe drives only 2, 4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"
- moved on the sheet: R1013, R1014

Commit message: review r4 item 4: the rail probe header moves to the sheet it observes
J1004 sat on mcu in a block of its own. Its own note said why, and named the
alternative: "power_rails is the alternative home." The captain has chosen it,
and it is the better one - the rails, their isolation links and their current
breaks are all on power_rails, and the header only observes them. It is J301
now, in block D, which already carries RAIL_PGOOD, D303 and TP308, the other
rail-observation parts. mcu loses a whole block rectangle.

The connector, its four rail flags, its ground rail and its note moved as one.
The first attempt moved the instance without its lib_symbol: KiCad loaded a
symbol with no pins, every wire on it collapsed, and the netlist showed all six
pads shorted onto one net. The lib_symbol travels with the part now, and mcu
drops the definition it no longer uses.

Also folded in: TEST_PLAN, DECISIONS, actuator-rev-testdebug (which listed this
move as an open item) and actuator-sch-mcu now say where these parts are. The
+5V5 rail keeps its name - the captain's own instruction calls it that - so the
block note carries the voltage instead, and TEST_PLAN's rail table says the name
is historical. Renaming it is a decision, not a tidy-up.

Round 4 complete: ERC 0/0 at severity-all, 409 components, 265 nets, zero
clearance findings on all ten sheets, zero misaligned ground rows, review pack
regenerated.

Co-Authored-By: Claude Opus 5 <noreply@anthropic.com>
Claude-Session: https://claude.ai/code/session_01PFWfwT8RZc8Zqn8vgZxV8j
Parts:
- removed J1004: PH1-06-UA, Amodo:Adam_Tech_PH1-06-UA, symbol Amodo_Connectors:Header_Male_6-way_1-row_Straight_2.54mm_THT
Other:
- note removed: "J RAIL PROBE HEADER (TEST_PLAN 4)"
- note removed: "One header to check every logic rail with a DMM during bring-up steps 2 and 3 of TEST_PLAN 5. The rails themselves, and their isolation links and current breaks, belong to power_rails - this header only observes them. 1 +5V 2 +3V3 3 +3V3A 4 GND 5 GND 6 GND +24V IS DELIBERATELY NOT ON THIS HEADER. 24 V next to 3.3 V on a 2.54 mm strip is one slip away from destroying the board; power_entry_24v alr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"
