File: hardware/kicad/faff2_cbs1/mcu.kicad_sch (KiCad schematic)
At the start: 62 parts, among them J1001 USB_C_Receptacle_USB2.0_16P, J1002 TSW-105-07-F-D, J1003 SAMTEC_SHF-107-01-L-D-SM, SW1001 PTS526, U1001 STM32H723VET6, U1002 USB3320C, U1003 SRAM 32Mb, U1004 MIC5365-1.8, Y1001 24MHz, Y1002 24MHz 18pF

Commit message: Hand tweaks by human
Parts:
- removed TP1003: 24MHZ, Amodo:TestPoint_Dual_D1.5mm_H1.0mm, symbol Amodo_Connectors:TestPointDual
- renumbered J1003 to J?
Other:
- moved on the sheet: R1013, R1014, R1015
