File: hardware/kicad/faff2_cbs1/mcu.kicad_sch (KiCad schematic)
At the start: 61 parts, among them J1001 USB_C_Receptacle_USB2.0_16P, J1002 TSW-105-07-F-D, SW1001 PTS526, U1001 STM32H723VET6, U1002 USB3320C, U1003 SRAM 32Mb, U1004 MIC5365-1.8, Y1001 24MHz, Y1002 24MHz 18pF

Commit message: review r5: the five verification findings, on top of the captain's state
Minimal deltas riding on his placement - nothing he moved is moved back unless
the finding was the move itself.

1. J603 and J1003 had lost their reference designators and both read "J?",
which merged them into a single netlist component: 17 nodes, pin numbers 3, 4,
5 and 10 twice, and only the 8510-4500PL's value and footprint, so the SAMTEC
SWD header had dropped out of the BOM altogether. Both references are set back
by hand, not by a blind re-annotate that would renumber other parts - and both
places that carry the name, the Reference property and the instance path's
(reference ...), because a sheet with those two disagreeing loads without
complaint and exports the old one. Proof: two distinct components now, J603
with 10 nodes on Amodo:8510-4500PL_LOGIC_TEST and J1003 with 14 on
Amodo:SAMTEC_SHF-107-01-L-D-SM, and the netlist export no longer warns about
annotation.

2. The +6V0 rename, completed again. c9d85d6 branched from 624bd13, one commit
before the rename, so the merge kept +6V0 on the net label, TP302's silkscreen
and the netlist net while restoring +5V5 in the title-block comment and four
note lines - leaving one note reading "+6V0 LMR33630 buck" two lines above "LDO
from +5V5". Those five, plus AGENTS.md, TEST_PLAN.md and
actuator-sch-power.md's current-state references, are back to +6V0. The
decisions-log history stays: DEC-P1 still explains why 5.5 V was chosen against
the TPS7A20's input maximum.

3. temp_sense: the ADS1120 block border sat at x=163.83, straight through
U701's body. The box is titled ADS1120 SUPPLIES AND SPI2 and U701 IS the
ADS1120, so the border goes to 151.13 - just left of the part, which is what
dragging it leftwards was reaching for - rather than back to 177.80.

4. power_rails: the two V24_LOGIC labels moved 1.27 mm left in the hand edit and
crossed the block border. The border moves instead, 13.97 -> 12.70, so his label
placement stands; 12.70 is the i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
Parts:
- gave numbers to parts that had none: 1
Changed lines of the file:
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@@
 		(on_board yes)
 		(dnp no)
-		(property "Reference" "J?"
+		(property "Reference" "J1003"
 			(at 445.77 104.14 0)
 			(effects
@@
 			(project "faff2_cbs1"
 				(path "/5edb00fd-45c9-5fe7-8d71-adbf38f38546/1d7ef20a-ceb5-5848-8c8d-02f7ee5f958f"
-					(reference "J?")
+					(reference "J1003")
 					(unit 1)
 				)
