File: hardware/kicad/faff2_cbs1/power_rails.kicad_sch (KiCad schematic)
At the start: 58 parts, among them U301 LMR33630, U302 ADPL42005, U303 ADPL42005, U304 LMR33630

Commit message: review r4 items 2,3,5,6,9: PGND, the frame boundary, and the U.FL connectors
Item 2, U304's PGND ground sitting on top of C318: the answer was already on
the sheet. U301 is the same regulator wired the same way, and its PGND ground
hangs 1.27 mm below the pin with its name clear above the VCC stub; U304's hung
6.35 mm down, which put it in C318's lane. Making it match U301 also closes both
of round 3's residual findings - power_rails is clear for the first time.

Item 3, the +5VA symbol outside the sheet boundary: the drawing area starts at
y=11.94, measured off a render, and the "+5VA" name's box ran 10.79..12.06 -
straddling it, inside the frame's ruler band. The whole excitation cluster drops
6.35 mm, the block box follows, and the feed keeps its long run and doglegs down
to the new row.

Item 9 is the same defect: temp_sense's PROBE 1 and CHANNEL 1 FILTER rectangles
start at y=11.43, half a millimetre above the drawing area. So do four of mcu's,
laid out to the same wrong value, so both sheets are fixed - every top edge to
12.70 and the titles under them to 13.34. Nothing on any sheet is above the
boundary now.

Item 5, FL501/FL502 -> J503/J504. The captain is right and there is no reason
that survives: they are Amodo_Connectors:CONUFL001-SMD, U.FL coaxial
connectors, with connector footprints, and the library symbol's own default
reference prefix is J. The FL prefix was an instance-level override
contradicting the part, and in IEEE-315 FL designates a filter. They sit in a
filter chain, which is the only reading that explains it. DEC-A14 records it.

Item 6, a concise pin-out beside J501. The full table was in the notes column
90 mm away; this is the five-line version directly under the connector, where
somebody landing a cable will look. Width is capped by the signal wires
dropping at x=48.26.

ERC 0/0 at severity-all; 408 components, 264 nets. The only netlist change is
item 5's re-designation - same nets, same members, new names.

Co-Authored-By: Claude Opus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
Changed lines of the file:
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@@
 	(wire
 		(pts
-			(xy 55.88 158.75) (xy 55.88 165.1)
+			(xy 55.88 158.75) (xy 55.88 160.02)
 		)
 		(stroke
@@
 	(symbol
 		(lib_id "Amodo_Symbols:GND")
-		(at 55.88 165.1 0)
+		(at 55.88 160.02 0)
 		(unit 1)
 		(exclude_from_sim no)
@@
 		(fields_autoplaced no)
 		(property "Reference" "#PWR327"
-			(at 55.88 165.1 0)
+			(at 55.88 160.02 0)
 			(effects
 				(font
@@
 		)
 		(property "Value" "GND"
-			(at 55.88 168.91 0)
+			(at 55.88 163.83 0)
 			(effects
 				(font
@@
 		)
 		(property "Footprint" ""
-			(at 55.88 165.1 0)
+			(at 55.88 160.02 0)
 			(effects
 				(font
@@
 		)
 		(property "Datasheet" ""
-			(at 55.88 165.1 0)
+			(at 55.88 160.02 0)
 			(effects
 				(font
@@
 		)
 		(property "Description" "Power symbol creates a global label with name \"GND\" , ground"
-			(at 55.88 165.1 0)
+			(at 55.88 160.02 0)
 			(effects
 				(font
@@
 		)
 		(property "SymLifecycle" "tested"
-			(at 55.88 165.1 0)
+			(at 55.88 160.02 0)
 			(effects
 				(font
@@
 		)
 		(property "ki_keywords" "global power"
-			(at 55.88 165.1 0)
+			(at 55.88 160.02 0)
 			(effects
 				(font

Commit message: review r4: the captain's two power answers - PG into RAIL_PGOOD, +5V5 to 6 V
A1. Both ADPL42005 power-good pins join DEC-P9's wired-AND. R317 and R318, 1 k
each like R315/R316, from each PG down to a local RAIL_PGOOD label - the idiom
the sheet already uses to reach that node three times. A dead 5 V rail is now
visible at D303 and TP308, which is the gap round 3 raised.

A2. +5V5 becomes 6.110 V nominal. The captain asked for 6.0 V - the
ADPL42005's characterised VIN = VOUT + 1 V point - or slightly above only if the
tolerance stack needs it to guarantee a 6.0 V minimum. It does: the LMR33630's
feedback reference is 0.985/1.000/1.015 V, +/-1.5% over the operating range, so
a 100k/20k divider gives 5.900/6.000/6.100 - nominal exactly on target, floor
100 mV short. 64.9k/12.7k gives 6.009/6.110/6.212 and the floor clears. Both
options and the arithmetic are in DEC-P10, along with what else moves: divider
impedance 122.1k to 77.6k so the 50 nA FB bias costs 3.2 mV, duty 0.255 at 24 V
in, caps still better than 2.5x derated, LDO dissipation 139 mW worst case.

Two traps on the way, both worth the tools that caught them. Hand-building the
new resistor block assembled its effects string with a str.replace on
"\t\t\t)", which also matched the font block's closing paren and put (hide yes)
inside it - KiCad answered "Failed to load schematic" and truncated the sheet to
349 components. The netlist component count is what caught it; ERC alone said
220 violations without saying why. New instances are cloned from an existing one
now. And set_lib_id alone left R303 and R304 carrying the OLD parts' mpn,
datasheet and description - a swap that looks right on the sheet and ships the
wrong part number to the BOM. sch_edit.sync_properties refreshes them from the
library, and both now read ERA-3AEB6492V and ERA-3AEB1272V.

ERC 0/0 at severity-all; 408 components, 264 nets; zero clearance findings. The
netlist change is exactly the two PG branches.

Co-Authored-By: Claude Opus 5 <norepl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
Parts:
- added R317, R318: 1k, Amodo:R_0603_1608Metric, symbol Amodo_Resistors:RES_TF_1k_0603
- R303: value 100k -> 64k9; symbol Amodo_Resistors:RES_TNF_100k_0603_0.1% -> Amodo_Resistors:RES_TNF_64.9k_0603_0.1%; gpn 667-ERA-3VEB1003V -> (none); mpn ERA-3VEB1003V -> ERA-3AEB6492V
- R304: value 22k1 -> 12k7; symbol Amodo_Resistors:RES_TNF_22.1k_0603_0.1% -> Amodo_Resistors:RES_TNF_12.7k_0603_0.1%; mpn RT0603BRD0722K1L -> ERA-3AEB1272V
Connections:
- net RAIL_PGOOD: now also R317.2, R318.2
- net at U303.7 (PG): now also R318.1
- net at U302.7 (PG): now also R317.1
- no-connect marks 2 -> 0
Other:
- note added: "6.0 V, not 5.0 V: it is the ADPL42005's own characterised VIN = VOUT + 1 V point, so the LDOs meet their noise and PSRR numbers on +5VA, which carries REQ-FF-04. R303/R304 are sized so the worst-case floor clears 6.0 V, not just the nominal: 6.009 / 6.110 / 6.212 V. Was 5.5 V while the TPS7A20's 6.0 V input maximum capped it."
- note added: "A. PRE-REGULATOR V24_LOGIC -> 6.0 V (LMR33630, 400 kHz)"
- note added: "BLOCK: power_rails - rail set and topology; answers OQ-02 and OQ-07 RAILS +6V0 LMR33630 buck from V24_LOGIC. Pre-regulator only, local to this sheet. +5V ADPL42005 LDO from +5V5. IKP11 read head (<65 mA plus RS-422 drive) and spare. +5VA ADPL42005 LDO from +5V5. ADS1235 / ADS1120 AVDD and the AFE 5 V excitation and reference chain, which lives in loadcell_afe - take it from +5VA, not +5V. +3V3 LM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"
- note removed: "5.5 V, not 5.0 V: it gives both ADPL42005 LDOs their dropout headroom. 500 mV covers the 325 mV worst-case dropout at 300 mA (Table 1); the part takes up to 20 V in, so 6.0 V no longer caps it."
- note removed: "A. PRE-REGULATOR V24_LOGIC -> 5.5 V (LMR33630, 400 kHz)"
- note removed: "BLOCK: power_rails - rail set and topology; answers OQ-02 and OQ-07 RAILS +5V5 LMR33630 buck from V24_LOGIC. Pre-regulator only, local to this sheet. +5V ADPL42005 LDO from +5V5. IKP11 read head (<65 mA plus RS-422 drive) and spare. +5VA ADPL42005 LDO from +5V5. ADS1235 / ADS1120 AVDD and the AFE 5 V excitation and reference chain, which lives in loadcell_afe - take it from +5VA, not +5V. +3V3 LM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"

Commit message: review r4 item 4: the rail probe header moves to the sheet it observes
J1004 sat on mcu in a block of its own. Its own note said why, and named the
alternative: "power_rails is the alternative home." The captain has chosen it,
and it is the better one - the rails, their isolation links and their current
breaks are all on power_rails, and the header only observes them. It is J301
now, in block D, which already carries RAIL_PGOOD, D303 and TP308, the other
rail-observation parts. mcu loses a whole block rectangle.

The connector, its four rail flags, its ground rail and its note moved as one.
The first attempt moved the instance without its lib_symbol: KiCad loaded a
symbol with no pins, every wire on it collapsed, and the netlist showed all six
pads shorted onto one net. The lib_symbol travels with the part now, and mcu
drops the definition it no longer uses.

Also folded in: TEST_PLAN, DECISIONS, actuator-rev-testdebug (which listed this
move as an open item) and actuator-sch-mcu now say where these parts are. The
+5V5 rail keeps its name - the captain's own instruction calls it that - so the
block note carries the voltage instead, and TEST_PLAN's rail table says the name
is historical. Renaming it is a decision, not a tidy-up.

Round 4 complete: ERC 0/0 at severity-all, 409 components, 265 nets, zero
clearance findings on all ten sheets, zero misaligned ground rows, review pack
regenerated.

Co-Authored-By: Claude Opus 5 <noreply@anthropic.com>
Claude-Session: https://claude.ai/code/session_01PFWfwT8RZc8Zqn8vgZxV8j
Parts:
- added J301: PH1-06-UA, Amodo:Adam_Tech_PH1-06-UA, symbol Amodo_Connectors:Header_Male_6-way_1-row_Straight_2.54mm_THT
Connections:
- net +3V3: now also J301.2
- net +3V3A: now also J301.3
- net +5V: now also J301.1
- net GND: now also J301.4, J301.5, J301.6
Other:
- note added: "D. ANALOG 3V3, RAIL POWER-GOOD, AND THE RAIL PROBE HEADER"
- note added: "RAIL PROBE HEADER (TEST_PLAN 4) One header to check every logic rail with a DMM during bring-up steps 2 and 3 of TEST_PLAN 5. It only observes: the rails, their isolation links and their current breaks are the rest of this sheet. 1 +5V 2 +3V3 3 +3V3A 4 GND 5 GND 6 GND +24V IS DELIBERATELY NOT ON THIS HEADER. 24 V next to 3.3 V on a 2.54 mm strip is one slip away from destroying the board; power_e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"
- note removed: "D. ANALOG 3V3 FOR THE ADC DIGITAL SUPPLIES, AND RAIL POWER-GOOD"

Commit message: review r4: finish the 6 V change - the rail is +6V0 everywhere
The captain is right that this was incomplete, not open. Raising the
pre-regulator to 6.110 V and leaving the net called +5V5 - with a note saying
the name was historical - left the label, the test point's silkscreen name and
half the sheet's text disagreeing with the voltage. That is worse than either
choice on its own: a rail whose name contradicts its value is a trap for whoever
reads the board next, and flagging it as a question did not make it safe.

+5V5 is a local label, not a library power symbol, so the rename touched
power_rails alone: no project-local symbol, no root-sheet pin, no other sheet.
Renamed on the drawing: the net label, TP302's silkscreen name, the title
block's one-line topology summary, the rail list in the block note, the per-rail
break list and the sequencing line. The "was 5.5 V" sentence came off the sheet
entirely - the drawing states the design as it is, and DEC-P10 carries the
history.

Swept in the docs: AGENTS.md's PWR_FLAG owner list, TEST_PLAN's rail table, and
actuator-sch-power.md's topology diagram, DEC-P1 heading, converter comparison
table and interface lists. DEC-P1's body still explains why 5.5 V was chosen
against the TPS7A20's input maximum, with a note at the top saying the rail's
name and voltage are now the ones in the heading - that history is deliberate.
No text outside the decisions log claims 5.5 V for this rail any more, and no
5V5 survives in any schematic or symbol file.

The netlist rename: /power_rails/+5V5 -> /power_rails/+6V0, membership identical
- C309.1, C312.1, R305.2, TP302.1, U302.5, U302.8, U303.5, U303.8. Verified as a
multiset compare of every net's node set, not by reading the diff.

ERC 0/0 at severity-all; 409 components, 265 nets; zero clearance findings, zero
misaligned ground rows; review pack regenerated.

Co-Authored-By: Claude Opus 5 <noreply@anthropic.com>
Claude-Session: https://claude.ai/code/session_01PFWfwT8RZc8Zqn8vgZxV8j
Parts:
- TP302: value +5V5 -> +6V0
Connections:
- net +5V5 renamed +6V0
Other:
- note added: "6.0 V, not 5.0 V: it is the ADPL42005's own characterised VIN = VOUT + 1 V point, so the LDOs meet their noise and PSRR numbers on +5VA, which carries REQ-FF-04. R303/R304 are sized so the worst-case floor clears 6.0 V, not just the nominal: 6.009 / 6.110 / 6.212 V. DEC-P10 has the stack."
- note added: "BLOCK: power_rails - rail set and topology; answers OQ-02 and OQ-07 RAILS +6V0 LMR33630 buck from V24_LOGIC, 6.110 V nominal. Pre-regulator only, local to this sheet. DEC-P10. +5V ADPL42005 LDO from +6V0. IKP11 read head (<65 mA plus RS-422 drive) and spare. +5VA ADPL42005 LDO from +6V0. ADS1235 / ADS1120 AVDD and the AFE 5 V excitation and reference chain, which lives in loadcell_afe - take it f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"
- note added: "PER RAIL (docs/TEST_PLAN.md 3.1) one 0R link that is BOTH the isolation link and the current-measurement break, a test point downstream of it, on a dual pad so a scope ground clips beside the probe. No test point sits on a feedback node: R305 +6V0, R306 +5V, R307 +5VA, R312 +3V3, FB301 +3V3A. Per-CONSUMER links are not here: every block takes the same global rail net, so per-block breaks would ne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"
- note removed: "6.0 V, not 5.0 V: it is the ADPL42005's own characterised VIN = VOUT + 1 V point, so the LDOs meet their noise and PSRR numbers on +5VA, which carries REQ-FF-04. R303/R304 are sized so the worst-case floor clears 6.0 V, not just the nominal: 6.009 / 6.110 / 6.212 V. Was 5.5 V while the TPS7A20's 6.0 V input maximum capped it."
- note removed: "BLOCK: power_rails - rail set and topology; answers OQ-02 and OQ-07 RAILS +6V0 LMR33630 buck from V24_LOGIC. Pre-regulator only, local to this sheet. +5V ADPL42005 LDO from +5V5. IKP11 read head (<65 mA plus RS-422 drive) and spare. +5VA ADPL42005 LDO from +5V5. ADS1235 / ADS1120 AVDD and the AFE 5 V excitation and reference chain, which lives in loadcell_afe - take it from +5VA, not +5V. +3V3 LM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"
- note removed: "PER RAIL (docs/TEST_PLAN.md 3.1) one 0R link that is BOTH the isolation link and the current-measurement break, a test point downstream of it, on a dual pad so a scope ground clips beside the probe. No test point sits on a feedback node: R305 +5V5, R306 +5V, R307 +5VA, R312 +3V3, FB301 +3V3A. Per-CONSUMER links are not here: every block takes the same global rail net, so per-block breaks would ne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"
Changed lines of the file:
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@@
 		(rev "0.2")
 		(company "Amodo Design")
-		(comment 1 "24 V -> 5V5 pre-reg -> +5V and +5VA; 24 V -> +3V3 -> +3V3A")
+		(comment 1 "24 V -> 6V0 pre-reg -> +5V and +5VA; 24 V -> +3V3 -> +3V3A")
 		(comment 2 "Per-rail isolation link / current break and test point")
 		(comment 3 "Rail set and topology answer OQ-02 / OQ-07")
@@
 		)
 	)
-	(label "+5V5"
+	(label "+6V0"
 		(at 196.85 63.5 0)
 		(effects
@@
 		)
 	)
-	(text "6.0 V, not 5.0 V: it is the ADPL42005's own\ncharacterised VIN = VOUT + 1 V point, so the LDOs\nmeet their noise and PSRR numbers on +5VA, which\ncarries REQ-FF-04.  R303/R304 are sized so the\nworst-case floor clears 6.0 V, not just the nominal:\n6.009 / 6.110 / 6.212 V.  Was 5.5 V while the\nTPS7A20's 6.0 V input maximum capped it."
+	(text "6.0 V, not 5.0 V: it is the ADPL42005's own\ncharacterised VIN = VOUT + 1 V point, so the LDOs\nmeet their noise and PSRR numbers on +5VA, which\ncarries REQ-FF-04.  R303/R304 are sized so the\nworst-case floor clears 6.0 V, not just the nominal:\n6.009 / 6.110 / 6.212 V.  DEC-P10 has the stack."
 		(exclude_from_sim no)
 		(at 20.32 105.41 0)
@@
 		)
 	)
-	(text "BLOCK: power_rails  -  rail set and topology; answers OQ-02 and OQ-07\n\nRAILS  +6V0   LMR33630 buck from V24_LOGIC. Pre-regulator only,\n              local to this sheet.\n       +5V    ADPL42005 LDO from +5V5. IKP11 read head (<65 mA plus\n              RS-422 drive) and spare.\n       +5VA   ADPL42005 LDO from +5V5. ADS1235 / ADS1120 AVDD and the\n              AFE 5 V excitation and reference chain, which lives in\n              loadcell_afe - take it from +5VA, not +5V.\n       +3V3   LMR33630 buck from V24_LOGIC. STM32, USB3320, DRV8323\n              logic, QSPI, EEPROM, RS-422 receiver, rotary encoder.\n              ~1.1 A worst case against a 3 A part.\n       +3V3A  ferrite-isolated from +3V3 for the ADC digital supplies.\n\nWHY A PRE-REGULATOR   The analog 5 V must be regulated separately from\n       the digital 5 V or the read head switching current lands on the\n       ADC supply, and an LDO needs headroom above 5 V to do it. One\n       buck at 6.0 V feeding two LDOs costs one converter and post-\n       regulates both 5 V rails. 400 kHz on both bucks: 3.3 V at\n       1.4 MHz would need a ~98 ns on-time, too close to the minimum."
+	(text "BLOCK: power_rails  -  rail set and topology; answers OQ-02 and OQ-07\n\nRAILS  +6V0   LMR33630 buck from V24_LOGIC, 6.110 V nominal.\n              Pre-regulator only, local to this sheet.  DEC-P10.\n       +5V    ADPL42005 LDO from +6V0. IKP11 read head (<65 mA plus\n              RS-422 drive) and spare.\n       +5VA   ADPL42005 LDO from +6V0. ADS1235 / ADS1120 AVDD and the\n              AFE 5 V excitation and reference chain, which lives in\n              loadcell_afe - take it from +5VA, not +5V.\n       +3V3   LMR33630 buck from V24_LOGIC. STM32, USB3320, DRV8323\n              logic, QSPI, EEPROM, RS-422 receiver, rotary encoder.\n              ~1.1 A worst case against a 3 A part.\n       +3V3A  ferrite-isolated from +3V3 for the ADC digital supplies.\n\nWHY A PRE-REGULATOR   The analog 5 V must be regulated separately from\n       the digital 5 V or the read head switching current lands on the\n       ADC supply, and an LDO needs headroom above 5 V to do it. One\n       buck at 6.0 V feeding two LDOs costs one converter and post-\n       regulates both 5 V rails. 400 kHz on both bucks: 3.3 V at\n       1.4 MHz would need a ~98 ns on-time, too close to the minimum."
 		(exclude_from_sim no)
 		(at 15.24 240.03 0)
@@
 		)
 	)
-	(text "PER RAIL (docs/TEST_PLAN.md 3.1)   one 0R link that is BOTH the\n       isolation link and the current-measurement break, a test point\n       downstream of it, on a dual pad so a scope ground clips beside\n       the probe. No test point sits on a feedback node:\n       R305 +5V5, R306 +5V, R307 +5VA, R312 +3V3, FB301 +3V3A.\n       Per-CONSUMER links are not here: every block takes the same\n       global rail net, so per-block breaks would need per-block rail\n       names and would break the frozen block contracts. A block that\n       wants one fits a 0R at its own supply entry, inside its sheet.\n\nSEQUENCING   None required. The shared EN divider (16.2 V rising) holds\n       both converters off until the 24 V input is real; the LDOs follow\n       +5V5 and +3V3A follows +3V3.\n\nINTERFACES   IN  V24_LOGIC <- power_entry_24v (owns its PWR_FLAG).\n       RAIL_PGOOD is open drain, the wired-AND of all four regulators\n       through R315 / R316 / R317 / R318. SHEET-LOCAL: LED D303, TP308\n       are its only consumers until OQ-07 allocates an MCU GPIO.\n       Global power nets produced here: +5V, +5VA, +3V3, +3V3A.\n       GND is board-wide, one net; power_entry_24v owns its PWR_FLAG.\n\nReasoning, part sizing and residual ERC:\n       docs/decisions/actuator-sch-power.md"
+	(text "PER RAIL (docs/TEST_PLAN.md 3.1)   one 0R link that is BOTH the\n       isolation link and the current-measurement break, a test point\n       downstream of it, on a dual pad so a scope ground clips beside\n       the probe. No test point sits on a feedback node:\n       R305 +6V0, R306 +5V, R307 +5VA, R312 +3V3, FB301 +3V3A.\n       Per-CONSUMER links are not here: every block takes the same\n       global rail net, so per-block breaks would need per-block rail\n       names and would break the frozen block contracts. A block that\n       wants one fits a 0R at its own supply entry, inside its sheet.\n\nSEQUENCING   None required. The shared EN divider (16.2 V rising) holds\n       both converters off until the 24 V input is real; the LDOs follow\n       +6V0 and +3V3A follows +3V3.\n\nINTERFACES   IN  V24_LOGIC <- power_entry_24v (owns its PWR_FLAG).\n       RAIL_PGOOD is open drain, the wired-AND of all four regulators\n       through R315 / R316 / R317 / R318. SHEET-LOCAL: LED D303, TP308\n       are its only consumers until OQ-07 allocates an MCU GPIO.\n       Global power nets produced here: +5V, +5VA, +3V3, +3V3A.\n       GND is board-wide, one net; power_entry_24v owns its PWR_FLAG.\n\nReasoning, part sizing and residual ERC:\n       docs/decisions/actuator-sch-power.md"
 		(exclude_from_sim no)
 		(at 204.47 240.03 0)
@@
 			)
 		)
-		(property "Value" "+5V5"
+		(property "Value" "+6V0"
 			(at 196.85 72.25 90)
 			(effects
