File: hardware/kicad/faff2_cbs1/ui_io.kicad_sch (KiCad schematic)
At the start: 40 parts, among them J901 BTN EXT, J902 SMA Jack, J903 J-LIM, SW901 PTS526, SW902 PTS526, SW903 PTS526, SW904 PTS526, U901 SN74LVC1G17, U902 SN74LVC1G11

Commit message: review: retire the last two pre-rotated passives, and the local library with them
The rotation rule is settled, so the two variants that predated it go the same
way as RES_TF_100R_0603_H did in round 4. R907 (39R) and R915 (0R) on ui_io move
to Amodo_Resistors:RES_TF_39R_0603 and RES_TF_0R_0603, rotated 90 with their
field angles compensated to 270; a render confirms both bodies horizontal with
horizontal reference and value, which is the condition the rule attaches.

The netlist is untouched because pin order is preserved: the _H variant has pin
1 at (0,0) and pin 2 at (5.08,0), and the house symbol at 90 degrees puts pin 1
at (X,Y) and pin 2 at (X+5.08,Y) - pin 1 on the left either way. Node sets are
identical across all 272 nets. What changed in the netlist is the libsource, and
the description string cached on each instance, which had said "horizontal
variant" and is now the house text; value and footprint were already the same
part number.

faff2_passives.kicad_sym held nothing else, so the file and its sym-lib-table
entry are deleted. AGENTS.md now says no pre-rotated variant exists, and
D-REV-07 - the decision that created the library - is marked superseded with the
residual it left ("the two horizontal resistors want to be house parts") closed:
they are house parts, and nothing is wanted upstream.

ERC 0/0 at severity-all; 408 components, 272 nets, node sets identical; zero
clearance findings; zero misaligned ground rows.

Co-Authored-By: Claude Opus 5 <noreply@anthropic.com>
Claude-Session: https://claude.ai/code/session_01PFWfwT8RZc8Zqn8vgZxV8j
Parts:
- R907: symbol faff2_passives:RES_TF_39R_0603_H -> Amodo_Resistors:RES_TF_39R_0603
- R915: symbol faff2_passives:RES_TF_0R_0603_H -> Amodo_Resistors:RES_TF_0R_0603
Other:
- moved on the sheet: R907, R915
Changed lines of the file:
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@@
 	)
 	(symbol
-		(lib_id "faff2_passives:RES_TF_39R_0603_H")
-		(at 184.15 25.4 0)
+		(lib_id "Amodo_Resistors:RES_TF_39R_0603")
+		(at 184.15 25.4 90)
 		(unit 1)
 		(exclude_from_sim no)
@@
 		(dnp no)
 		(property "Reference" "R907"
-			(at 186.69 22.86 0)
+			(at 186.69 22.86 270)
 			(effects
 				(font
@@
 		)
 		(property "Value" "39R"
-			(at 186.69 27.94 0)
+			(at 186.69 27.94 270)
 			(effects
 				(font
@@
 		)
 		(property "Footprint" "Amodo:R_0603_1608Metric"
-			(at 184.15 25.4 0)
+			(at 184.15 25.4 270)
 			(effects
 				(font
@@
 		)
 		(property "Datasheet" "https://www.mouser.co.uk/datasheet/2/315/AOA0000C304-1149620.pdf"
-			(at 184.15 25.4 0)
+			(at 184.15 25.4 270)
 			(effects
 				(font
@@
 		)
 		(property "Description" "SMD Thick Film Resistor 39R 0603 1% 100mW"
-			(at 184.15 25.4 0)
+			(at 184.15 25.4 270)
 			(effects
 				(font
@@
 		)
 		(property "mpn" "ERJ-3EKF39R0V"
-			(at 184.15 25.4 0)
+			(at 184.15 25.4 270)
 			(effects
 				(font
@@
 		)
 		(property "gpn" "GPR060339R"
-			(at 184.15 25.4 0)
+			(at 184.15 25.4 270)
 			(effects
 				(font
@@
 		)
 		(property "SymLifecycle" "draft"
-			(at 184.15 25.4 0)
+			(at 184.15 25.4 270)
 			(effects
 				(font
@@
 	)
 	(symbol
-		(lib_id "faff2_passives:RES_TF_0R_0603_H")
-		(at 190.5 194.31 0)
+		(lib_id "Amodo_Resistors:RES_TF_0R_0603")
+		(at 190.5 194.31 90)
 		(unit 1)
 		(exclude_from_sim no)
@@
 		(dnp no)
 		(property "Reference" "R915"
-			(at 193.04 192.28 0)
+			(at 193.04 192.28 270)
 			(effects
 				(font
@@
 		)
 		(property "Value" "0R"
-			(at 193.04 196.6 0)
+			(at 193.04 196.6 270)
 			(effects
 				(font
@@
 		)
 		(property "Footprint" "Amodo:R_0603_1608Metric"
-			(at 190.5 194.31 0)
+			(at 190.5 194.31 270)
 			(effects
 				(font
@@
 			)
 		)
-		(property "Datasheet" "~"
-			(at 190.5 194.31 0)
+		(property "Datasheet" ""
+			(at 190.5 194.31 270)
 			(effects
 				(font
@@
 		)
 		(property "Description" "SMD Thick Film Resistor 0R 0603 1% 100mW"
-			(at 190.5 194.31 0)
+			(at 190.5 194.31 270)
 			(effects
 				(font
@@
 		)
 		(property "mpn" "RC0603FR-070RL"
-			(at 190.5 194.31 0)
+			(at 190.5 194.31 270)
 			(effects
 				(font
@@
 		)
 		(property "SymLifecycle" "tested"
-			(at 190.5 194.31 0)
+			(at 190.5 194.31 270)
 			(effects
 				(font
